File: base/base.kicad_pcb (KiCad board)
At the start: 2 copper layers, 175.4 x 112.3 mm, 136 parts, among them J1 24V_PINOUTS_ARM, J10 12V_BUCK_PINOUTS_ARM, J11 12V_BUCK_PINOUTS_ARM, J12 12V_BUCK_PINOUTS_ARM, J14 JETSON_POWER, J15 12V_BUCK_PINOUTS_ARM, J18 BASE_POWER_IN, J19 BuckOut, J2 Conn_01x20_Pin, J20 BatteryIn2, J21 KSMain2, J22 USB_C_Receptacle_USB2.0_14P, J23 MDDPOWER5, J24 MDDPOWER7, J25 MDDPOWER8, J26 MDDPOWER6, J3 BASE_KILL_SWITCH, J4 5VISO_IN, J5 Conn_01x20_Pin, J6 BASE_KILL_SWITCH, J7 12V_BUCK_PINOUTS_ARM, J8 24V_PINOUTS_ARM, J9 12V_BUCK_PINOUTS_ARM, U10 USBLC6-4SC6, U11 USBLC6-4SC6, U13 USBLC6-4SC6, U14 USBLC6-4SC6, U16 USBLC6-4SC6, U17 USBLC6-4SC6, U18 USBLC6-4SC6, U2 USBLC6-4SC6, U23 6N137, U24 6N137, U25 6N137, U26 6N137, U27 6N137, U28 6N137, U29 6N137, U3 USBLC6-4SC6, U30 6N137, U31 6N137, U32 6N137, U33 6N137, U34 6N137, U36 6N137, U37 6N137

Commit message: fixed labels
Parts:
- added BNO1: Polyfuse, Fuse:Fuse_0603_1608Metric_Pad1.05x0.95mm_HandSolder, F.Cu at (125.7, 150.3)
- added D2: RB160M (1 A diode), Diode_SMD:D_SOD-123F, F.Cu at (243.7, 151.1)
- added FB1: FerriteBead, Inductor_SMD:L_0805_2012Metric_Pad1.15x1.40mm_HandSolder, F.Cu at (57.4, 81.3)
- added J13: Conn_01x20_Pin, Connector_PinHeader_2.54mm:PinHeader_1x20_P2.54mm_Vertical, F.Cu at (201.9, 130.8)
- added J16: Conn_01x20_Pin, Connector_PinHeader_2.54mm:PinHeader_1x20_P2.54mm_Vertical, F.Cu at (234.9, 179.1)
- added MainFuse1: Fuse, Fuse:Fuseholder_Littelfuse_445_030_series_5x30mm, F.Cu at (167.4, 212.1)
- added MotorController1: STM32F411_BP, ROBO:STM32F411-BP, F.Cu at (157.5, 168.9)
- added MotorController2: STM32F411_BP, ROBO:STM32F411-BP, F.Cu at (218.4, 153.7)
- added STMFuse1: Polyfuse, Fuse:Fuse_0603_1608Metric_Pad1.05x0.95mm_HandSolder, F.Cu at (241.3, 109.6)
- added U1: UA741CP, UA741CP:DIP794W45P254L959H508Q8, F.Cu at (266.3, 162.6)
- added U15: BNO055, ROBO:7_semi_BNO055, F.Cu at (137.3, 109.0)
- added U9: ~, ROBO:WRB0505S-3WR3, F.Cu at (245.5, 139.4)
- J22: footprint Connector_AMASS:AMASS_XT60PW-M_1x02_P7.20mm_Horizontal -> Connector_USB:USB_C_Receptacle_GCT_USB4105-xx-A_16P_TopMnt_Horizontal
- STMCap1: footprint Connector_Phoenix_SPT:PhoenixContact_SPT_1.5_9-H-3.5_1x09_P3.5mm_Horizontal -> Capacitor_SMD:C_0805_2012Metric
- moved H6 352.1 mm to (3.50, 335.5)
- moved H5 329.2 mm to (170.0, 335.5)
- moved J18 327.0 mm to (278.1, 152.4), turned to -90 degrees
- moved H8 323.2 mm to (3.50, 232.0)
- moved J19 318.5 mm to (278.1, 170.2), turned to -90 degrees
- moved H7 315.4 mm to (170.0, 232.0)
- moved J20 311.9 mm to (278.1, 188.0), turned to -90 degrees
- moved J21 307.1 mm to (278.1, 205.7), turned to -90 degrees
- moved J10 293.2 mm to (213.6, 199.7), turned to 180 degrees
- moved J11 277.3 mm to (278.1, 82.5), turned to -90 degrees
- moved J9 273.5 mm to (235.6, 93.6)
- moved J12 266.3 mm to (278.1, 100.3), turned to -90 degrees
- moved J14 257.3 mm to (278.1, 118.1), turned to -90 degrees
- moved J15 249.8 mm to (278.1, 134.6), turned to -90 degrees
- moved J2 221.7 mm to (134.6, 184.2), turned to 90 degrees
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Other:
- board size 175.4 x 112.3 mm -> 217.2 x 157.5 mm

Commit message: suggested corrections made
Parts:
- removed U13, U14, U16, U17: USBLC6-4SC6, Package_TO_SOT_SMD:SOT-23-6
- added J17: BuckOut, Connector_AMASS:AMASS_XT60PW-M_1x02_P7.20mm_Horizontal, F.Cu at (347.9, 221.6)
- added J27: BuckIn, Connector_AMASS:AMASS_XT60PW-M_1x02_P7.20mm_Horizontal, F.Cu at (265.2, 200.1)
- added J28: BuckOut, Connector_AMASS:AMASS_XT60PW-M_1x02_P7.20mm_Horizontal, F.Cu at (248.6, 200.2)
- added J29: BuckIn, Connector_AMASS:AMASS_XT60PW-M_1x02_P7.20mm_Horizontal, F.Cu at (231.1, 200.2)
- J18: value BASE_POWER_IN -> EXTRA_PORT
- J19: value BuckOut -> KSMain2
- J4: value 5VISO_IN -> EXTRA_PORT
- moved U10 138.6 mm to (115.7, 164.1)
- moved R60 122.0 mm to (175.8, 136.7), turned to 180 degrees
- moved R68 121.7 mm to (184.4, 136.7), turned to 180 degrees
- moved R61 109.9 mm to (175.8, 129.5), turned to 180 degrees
- moved R69 109.1 mm to (184.4, 129.0), turned to 180 degrees
- moved R20 98.0 mm to (204.7, 96.0)
- moved R21 98.0 mm to (204.7, 101.1)
- moved R4 98.0 mm to (199.6, 96.0)
- moved R46 98.0 mm to (204.7, 106.2)
- moved R47 98.0 mm to (204.7, 106.2)
- moved R48 98.0 mm to (204.7, 111.3)
- moved R49 98.0 mm to (204.7, 111.3)
- moved R50 98.0 mm to (204.7, 116.3)
- moved R52 98.0 mm to (209.8, 96.0)
- moved R53 98.0 mm to (209.8, 101.1)
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Connections:
- net 12V_OUT_ARM renamed 12VOUT
- C2 pad 1: 5VIn -> 5VOut
- Encoder1 pad 1: 5VIn -> 5VOut
- Encoder1Capacitor1 pad 1: 5VIn -> 5VOut
- Encoder1Capacitor2 pad 1: 5VIn -> 5VOut
- Encoder1Capacitor3 pad 1: 5VIn -> 5VOut
- Encoder2 pad 1: 5VIn -> 5VOut
- Encoder3 pad 1: 5VIn -> 5VOut
- J13 pad 19: GND -> GND1
- J16 pad 19: GND -> GND1
- J16 pad 20: 5VOut -> STM5V_ISO
- L2 pad 1: 5VIn -> 5VOut
- MotorController2 pad 1: 5VOut -> STM5V_ISO
- MotorController2 pad 2: GND -> GND1
- MotorController2 pad 39: GND -> GND1
- U10 pad 2: Earth -> GND
- U11 pad 2: Earth -> GND
- U2 pad 2: Earth -> GND
- U3 pad 2: Earth -> GND
Other:
- board size 217.2 x 157.5 mm -> 217.2 x 148.3 mm

Commit message: dff
Parts:
- removed R46, R47, R48, R49, R54, R55, R56, R57, R62, R63, R64, R65, R71, R72: 4.7k, Resistor_SMD:R_0805_2012Metric_Pad1.20x1.40mm_HandSolder
- added STMFuse2: Polyfuse, Fuse:Fuse_0603_1608Metric_Pad1.05x0.95mm_HandSolder, F.Cu at (182.5, 134.6)
- BNOCapacitor1, C2, C20, C21, C22, C23, C24, C25, C26, C27, C28, C29, C3, C30, C31, C35, C36, C5, C7, C9, Encoder1Capacitor1, Encoder1Capacitor2, Encoder1Capacitor3: footprint Capacitor_SMD:C_0805_2012Metric_Pad1.18x1.45mm_HandSolder -> Capacitor_SMD:C_0201_0603Metric
- BNOLED1, Battery_Indication2, STMLED1: footprint LED_SMD:LED_0805_2012Metric_Pad1.15x1.40mm_HandSolder -> LED_SMD:LED_0201_0603Metric
- FB1: footprint Inductor_SMD:L_0805_2012Metric_Pad1.15x1.40mm_HandSolder -> PCM_Inductor_SMD_Handsoldering_AKL:L_CommonModeChoke_Coilcraft_0603USB
- J1, J15: footprint Connector_AMASS:AMASS_XT60PW-M_1x02_P7.20mm_Horizontal -> Connector_JST:JST_XH_B2B-XH-A_1x02_P2.50mm_Vertical
- J10, J11, J12, J14, J17, J18, J19, J20, J21, J23, J24, J25, J26, J27, J28, J29, J3, J4, J6, J7, J8, J9: footprint Connector_AMASS:AMASS_XT60PW-M_1x02_P7.20mm_Horizontal -> Connector_AMASS:AMASS_XT60-M_1x02_P7.20mm_Vertical
- L2: footprint Inductor_SMD:L_0805_2012Metric_Pad1.05x1.20mm_HandSolder -> PCM_Inductor_SMD_Handsoldering_AKL:L_0603_1608Metric_Pad1.05x0.95mm
- MainLED1: footprint LED_THT:LED_D3.0mm -> LED_SMD:LED_0201_0603Metric
- R1, R10, R11, R18, R19, R20, R21, R22, R23, R24, R25, R26, R27, R28, R29, R30, R4, R50, R51, R52, R53, R58, R59, R60, R61, R66, R67, R68, R69, R7, R73, R74, R8, R9: footprint Resistor_SMD:R_0805_2012Metric_Pad1.20x1.40mm_HandSolder -> PCM_4ms_Resistor:R_0603
- STMCap1: footprint Capacitor_SMD:C_0805_2012Metric -> Capacitor_SMD:C_0201_0603Metric
- moved H6 270.0 mm to (78.7, 76.2)
- moved H8 262.2 mm to (264.2, 203.2)
- moved C22 229.0 mm to (94.3, 191.0)
- moved C23 209.3 mm to (115.5, 178.3)
- moved C30 196.9 mm to (96.4, 157.0)
- moved C27 188.4 mm to (113.0, 168.7)
- moved C31 182.5 mm to (114.1, 149.9)
- moved H7 182.0 mm to (264.2, 76.2)
- moved J17 177.0 mm to (245.2, 77.5), turned to 0 degrees
- moved C35 174.3 mm to (97.7, 139.7)
- moved Battery_Indication2 164.8 mm to (120.6, 189.5)
- moved 1.5k1 162.5 mm to (173.7, 189.0), turned to 180 degrees
- moved C28 161.6 mm to (168.0, 147.3)
- moved C36 160.4 mm to (116.0, 133.6)
- moved H5 159.3 mm to (81.3, 203.2)
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Connections:
- BNO1 pad 1: 5V -> STM5V_ISO_IN
- H5 pad 1: Chassis -> GND
- H6 pad 1: Chassis -> GND
- H7 pad 1: Chassis -> GND
- H8 pad 1: Chassis -> GND
- J13 pad 19: GND1 -> GND
- J16 pad 19: GND1 -> GND
- J16 pad 20: STM5V_ISO -> 5VOut
- J5 pad 20: STM5V_ISO -> STM5V_ISO_IN
- MotorController1 pad 1: STM5V_ISO -> STM5V_ISO_IN
- MotorController2 pad 1: STM5V_ISO -> 5VOut
- MotorController2 pad 2: GND1 -> GND
- MotorController2 pad 39: GND1 -> GND
- R1 pad 2: 3V3 -> 5VOut
- R22 pad 1: 3V3 -> 5VOut
- R23 pad 2: 3V3 -> 5VOut
- R24 pad 1: 3V3 -> 5VOut
- R25 pad 2: 3V3 -> 5VOut
- R26 pad 1: 3V3 -> 5VOut
- R27 pad 1: 3V3 -> 5VOut
- R28 pad 2: 3V3 -> 5VOut
- STMFuse1 pad 1: 5V -> STM5V_ISO_IN
- U10 pad 5: 3V3M -> 5VOut
- U11 pad 5: 3V3M -> 5VOut
- U18 pad 5: 3V3S -> 5VOut
- U2 pad 5: 3V3S -> 5VOut
- U23 pad 2: Net-(U23-A) -> 5VIn
- U24 pad 2: Net-(U24-A) -> 5VIn
- U25 pad 2: Net-(U25-A) -> STM5V_ISO
- U26 pad 2: Net-(U26-A) -> STM5V_ISO
- U27 pad 2: Net-(U27-A) -> 5VIn
- U28 pad 2: Net-(U28-A) -> 5VIn
- U29 pad 2: Net-(U29-A) -> STM5V_ISO
- U3 pad 5: 3V3S -> 5VOut
- U30 pad 2: Net-(U30-A) -> STM5V_ISO
- U31 pad 2: Net-(U31-A) -> 5VIn
- U32 pad 2: Net-(U32-A) -> 5VIn
- U33 pad 2: Net-(U33-A) -> STM5V_ISO
- U34 pad 2: Net-(U34-A) -> STM5V_ISO
- U36 pad 2: Net-(U36-A) -> STM5V_ISO
- U37 pad 2: Net-(U37-A) -> STM5V_ISO
Other:
- board size 217.2 x 148.3 mm -> 198.1 x 138.2 mm
