File: base/base.kicad_sch (KiCad schematic)
At the start: 49 parts, among them J1 24V_PINOUTS_ARM, J10 12V_BUCK_PINOUTS_ARM, J11 12V_BUCK_PINOUTS_ARM, J12 12V_BUCK_PINOUTS_ARM, J14 JETSON_POWER, J15 12V_BUCK_PINOUTS_ARM, J18 BASE_POWER_IN, J19 BuckOut, J2 Conn_01x20_Pin, J20 BatteryIn2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

Commit message: fixed labels
Parts:
- added J13, J16: Conn_01x20_Pin, Connector_PinHeader_2.54mm:PinHeader_1x20_P2.54mm_Vertical, symbol Connector:Conn_01x20_Pin
- added J17, J28: BuckOut, Connector_AMASS:AMASS_XT60PW-M_1x02_P7.20mm_Horizontal, symbol XT60-M:XT60-M
- added J27, J29: BuckIn, Connector_AMASS:AMASS_XT60PW-M_1x02_P7.20mm_Horizontal, symbol XT60-M:XT60-M
- added MotorController2: STM32F411_BP, ROBO:STM32F411-BP, symbol RM_Footprints:STM32F411-BlackPill
- J22: footprint Connector_AMASS:AMASS_XT60PW-M_1x02_P7.20mm_Horizontal -> Connector_USB:USB_C_Receptacle_GCT_USB4105-xx-A_16P_TopMnt_Horizontal
Connections:
- net 12VOUT_ARM: now also J15.P (POS)
- net 24V: now also J29.P (POS)
- net 24VOUT_ARM: now also J1.P (POS)
- net 5VOut: now also J16.20 (Pin_20), J28.P (POS), MotorController2.1 (5V)
- net GND: now also J13.19 (Pin_19), J16.19 (Pin_19), J17.N (NEG), J27.N (NEG), J28.N (NEG), J29.N (NEG), MotorController2.2 (GND), MotorController2.39 (GND)
- net 12Vin_ARM renamed 12VOUT
- net 12VOUT: now also J17.P (POS); no longer J15.P (POS)
- net 24Vin_ARM: no longer names the net of J8.N (NEG)
- net 24Vin_ARM: no longer J1.P (POS)
- new net: J13.1 (Pin_1), MotorController2.21 (PB12)
- new net: J13.10 (Pin_10), MotorController2.30 (PA15)
- new net: J13.11 (Pin_11), MotorController2.31 (PB3)
- new net: J13.12 (Pin_12), MotorController2.32 (PB4)
- new net: J13.13 (Pin_13), MotorController2.33 (PB5)
- new net: J13.14 (Pin_14), MotorController2.34 (PB6)
- new net: J13.15 (Pin_15), MotorController2.35 (PB7)
- new net: J13.16 (Pin_16), MotorController2.36 (PB8)
- new net: J13.17 (Pin_17), MotorController2.37 (PB9)
- new net: J13.18 (Pin_18), MotorController2.38 (5V)
- new net: J13.2 (Pin_2), MotorController2.22 (PB13)
- new net: J13.20 (Pin_20), MotorController2.40 (3V3)
- new net: J13.3 (Pin_3), MotorController2.23 (PB14)
- new net: J13.4 (Pin_4), MotorController2.24 (PB15)
- new net: J13.5 (Pin_5), MotorController2.25 (PA8)
- new net: J13.6 (Pin_6), MotorController2.26 (PA9)
- new net: J13.7 (Pin_7), MotorController2.27 (PA10)
- new net: J13.8 (Pin_8), MotorController2.28 (PA11)
- new net: J13.9 (Pin_9), MotorController2.29 (PA12)
- new net: J16.1 (Pin_1), MotorController2.20 (VBat)
- new net: J16.10 (Pin_10), MotorController2.11 (PA4)
- new net: J16.11 (Pin_11), MotorController2.10 (PA5)
- new net: J16.12 (Pin_12), MotorController2.9 (PA6)
- new net: J16.13 (Pin_13), MotorController2.8 (PA7)
- new net: J16.14 (Pin_14), MotorController2.7 (PB0)
- new net: J16.15 (Pin_15), MotorController2.6 (PB1)
- new net: J16.16 (Pin_16), MotorController2.5 (PB2)
- new net: J16.17 (Pin_17), MotorController2.4 (PB10)
- new net: J16.18 (Pin_18), MotorController2.3 (3V3)
- new net: J16.2 (Pin_2), MotorController2.19 (PC13)
- new net: J16.3 (Pin_3), MotorController2.18 (PC14)
- new net: J16.4 (Pin_4), MotorController2.17 (PC15)
- new net: J16.5 (Pin_5), MotorController2.16 (RST)
- new net: J16.6 (Pin_6), MotorController2.15 (PA0)
- new net: J16.7 (Pin_7), MotorController2.14 (PA1)
- new net: J16.8 (Pin_8), MotorController2.13 (PA2)
- new net: J16.9 (Pin_9), MotorController2.12 (PA3)
Other:
- note added: "12V BUCK"
- note added: "5V BUCK"
- note added: "BATTERY PLUGIN"
- moved on the sheet: J10, J11, J12, J24, J25, J3, J6, J9, MotorController1, U13, U14, U16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

Commit message: fixed labels
Parts:
- J18: value BASE_POWER_IN -> EXTRA_PORT
Changed lines of the file:
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@@
 			)
 		)
-		(property "Value" "BASE_POWER_IN"
+		(property "Value" "EXTRA_PORT"
 			(at 227.965 76.835 0)
 			(effects

Commit message: suggested corrections made
Parts:
- removed U13, U14, U16, U17: USBLC6-4SC6, Package_TO_SOT_SMD:SOT-23-6, symbol Power_Protection:USBLC6-4SC6
- J1, J15: footprint Connector_AMASS:AMASS_XT60PW-M_1x02_P7.20mm_Horizontal -> Connector_JST:JST_XH_B2B-XH-A_1x02_P2.50mm_Vertical
- J19: value BuckOut -> KSMain2
- J4: value 5VISO_IN -> EXTRA_PORT
Connections:
- net 3V3S is gone; now on net 5VOut: U18.5 (VBUS)
- net 24V: now also J27.P (POS); no longer J29.P (POS)
- net 24VIn: now also J29.P (POS), J4.P (POS)
- net 24V_BATTERY_IN: now also J19.P (POS)
- net 3V3: no longer R1.2, R22.1, R23.2, R24.1, R25.2, R26.1, R27.1, R28.2
- net 5VIn: no longer Encoder1.1 (Pin_1), Encoder2.1 (Pin_1), Encoder3.1 (Pin_1), J4.P (POS)
- net 5VOut: now also Encoder1.1 (Pin_1), Encoder2.1 (Pin_1), Encoder3.1 (Pin_1), R1.2, R22.1, R23.2, R24.1, R25.2, R26.1, R27.1, R28.2; no longer J19.P (POS)
- net GND: no longer J19.N (NEG)
- net STM5V_ISO: no longer J5.20 (Pin_20), MotorController1.1 (5V)
- net 24VIn_Jetson renamed 24V_JETSON_IN
- net 24V_JETSON_IN: now also J19.N (NEG)
- new net STM5V_ISO_IN: J5.20 (Pin_20), MotorController1.1 (5V)
Other:
- note removed: "TVS DIODE"

Commit message: added 0603 footprint
Parts:
- FB1: footprint Inductor_SMD:L_0805_2012Metric_Pad1.15x1.40mm_HandSolder -> PCM_Inductor_SMD_Handsoldering_AKL:L_CommonModeChoke_Coilcraft_0603USB
- R1, R22, R23, R24, R25, R26, R27, R28, R29, R30: footprint Resistor_SMD:R_0805_2012Metric_Pad1.20x1.40mm_HandSolder -> PCM_4ms_Resistor:R_0603
Changed lines of the file:
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@@
 			)
 		)
-		(property "Footprint" "Resistor_SMD:R_0805_2012Metric_Pad1.20x1.40mm_HandSolder"
+		(property "Footprint" "PCM_4ms_Resistor:R_0603"
 			(at 213.614 221.869 90)
 			(effects
@@
 			)
 		)
-		(property "Footprint" "Resistor_SMD:R_0805_2012Metric_Pad1.20x1.40mm_HandSolder"
+		(property "Footprint" "PCM_4ms_Resistor:R_0603"
 			(at 213.614 219.329 90)
 			(effects
@@
 			)
 		)
-		(property "Footprint" "Resistor_SMD:R_0805_2012Metric_Pad1.20x1.40mm_HandSolder"
+		(property "Footprint" "PCM_4ms_Resistor:R_0603"
 			(at 107.95 179.705 0)
 			(effects
@@
 			)
 		)
-		(property "Footprint" "Resistor_SMD:R_0805_2012Metric_Pad1.20x1.40mm_HandSolder"
+		(property "Footprint" "PCM_4ms_Resistor:R_0603"
 			(at 106.68 140.335 0)
 			(effects
@@
 			)
 		)
-		(property "Footprint" "Resistor_SMD:R_0805_2012Metric_Pad1.20x1.40mm_HandSolder"
+		(property "Footprint" "PCM_4ms_Resistor:R_0603"
 			(at 136.525 129.54 0)
 			(effects
@@
 			)
 		)
-		(property "Footprint" "Resistor_SMD:R_0805_2012Metric_Pad1.20x1.40mm_HandSolder"
+		(property "Footprint" "PCM_4ms_Resistor:R_0603"
 			(at 106.68 128.905 0)
 			(effects
@@
 			)
 		)
-		(property "Footprint" "Inductor_SMD:L_0805_2012Metric_Pad1.15x1.40mm_HandSolder"
+		(property "Footprint" "PCM_Inductor_SMD_Handsoldering_AKL:L_CommonModeChoke_Coilcraft_0603USB"
 			(at 174.752 255.905 90)
 			(effects
@@
 			)
 		)
-		(property "Footprint" "Resistor_SMD:R_0805_2012Metric_Pad1.20x1.40mm_HandSolder"
+		(property "Footprint" "PCM_4ms_Resistor:R_0603"
 			(at 107.95 160.655 0)
 			(effects
@@
 			)
 		)
-		(property "Footprint" "Resistor_SMD:R_0805_2012Metric_Pad1.20x1.40mm_HandSolder"
+		(property "Footprint" "PCM_4ms_Resistor:R_0603"
 			(at 107.95 168.275 0)
 			(effects
@@
 			)
 		)
-		(property "Footprint" "Resistor_SMD:R_0805_2012Metric_Pad1.20x1.40mm_HandSolder"
+		(property "Footprint" "PCM_4ms_Resistor:R_0603"
 			(at 107.95 149.225 0)
 			(effects
@@
 			)
 		)
-		(property "Footprint" "Resistor_SMD:R_0805_2012Metric_Pad1.20x1.40mm_HandSolder"
+		(property "Footprint" "PCM_4ms_Resistor:R_0603"
 			(at 136.525 140.97 0)
 			(effects

Commit message: dff
Parts:
- J10, J11, J12, J14, J17, J18, J19, J20, J21, J23, J24, J25, J26, J27, J28, J29, J3, J4, J6, J7, J8, J9: footprint Connector_AMASS:AMASS_XT60PW-M_1x02_P7.20mm_Horizontal -> Connector_AMASS:AMASS_XT60-M_1x02_P7.20mm_Vertical
Changed lines of the file:
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@@
 			)
 		)
-		(property "Footprint" "Connector_AMASS:AMASS_XT60PW-M_1x02_P7.20mm_Horizontal"
+		(property "Footprint" "Connector_AMASS:AMASS_XT60-M_1x02_P7.20mm_Vertical"
 			(at 275.59 160.655 0)
 			(effects
@@
 			)
 		)
-		(property "Footprint" "Connector_AMASS:AMASS_XT60PW-M_1x02_P7.20mm_Horizontal"
+		(property "Footprint" "Connector_AMASS:AMASS_XT60-M_1x02_P7.20mm_Vertical"
 			(at 349.25 74.93 0)
 			(effects
@@
 			)
 		)
-		(property "Footprint" "Connector_AMASS:AMASS_XT60PW-M_1x02_P7.20mm_Horizontal"
+		(property "Footprint" "Connector_AMASS:AMASS_XT60-M_1x02_P7.20mm_Vertical"
 			(at 342.265 144.78 0)
 			(effects
@@
 			)
 		)
-		(property "Footprint" "Connector_AMASS:AMASS_XT60PW-M_1x02_P7.20mm_Horizontal"
+		(property "Footprint" "Connector_AMASS:AMASS_XT60-M_1x02_P7.20mm_Vertical"
 			(at 229.87 143.51 0)
 			(effects
@@
 			)
 		)
-		(property "Footprint" "Connector_AMASS:AMASS_XT60PW-M_1x02_P7.20mm_Horizontal"
+		(property "Footprint" "Connector_AMASS:AMASS_XT60-M_1x02_P7.20mm_Vertical"
 			(at 226.06 85.09 0)
 			(effects
@@
 			)
 		)
-		(property "Footprint" "Connector_AMASS:AMASS_XT60PW-M_1x02_P7.20mm_Horizontal"
+		(property "Footprint" "Connector_AMASS:AMASS_XT60-M_1x02_P7.20mm_Vertical"
 			(at 318.77 86.995 0)
 			(effects
@@
 			)
 		)
-		(property "Footprint" "Connector_AMASS:AMASS_XT60PW-M_1x02_P7.20mm_Horizontal"
+		(property "Footprint" "Connector_AMASS:AMASS_XT60-M_1x02_P7.20mm_Vertical"
 			(at 295.91 37.465 0)
 			(effects
@@
 			)
 		)
-		(property "Footprint" "Connector_AMASS:AMASS_XT60PW-M_1x02_P7.20mm_Horizontal"
+		(property "Footprint" "Connector_AMASS:AMASS_XT60-M_1x02_P7.20mm_Vertical"
 			(at 226.06 72.39 0)
 			(effects
@@
 			)
 		)
-		(property "Footprint" "Connector_AMASS:AMASS_XT60PW-M_1x02_P7.20mm_Horizontal"
+		(property "Footprint" "Connector_AMASS:AMASS_XT60-M_1x02_P7.20mm_Vertical"
 			(at 231.775 104.775 0)
 			(effects
@@
 			)
 		)
-		(property "Footprint" "Connector_AMASS:AMASS_XT60PW-M_1x02_P7.20mm_Horizontal"
+		(property "Footprint" "Connector_AMASS:AMASS_XT60-M_1x02_P7.20mm_Vertical"
 			(at 342.265 158.115 0)
 			(effects
@@
 			)
 		)
-		(property "Footprint" "Connector_AMASS:AMASS_XT60PW-M_1x02_P7.20mm_Horizontal"
+		(property "Footprint" "Connector_AMASS:AMASS_XT60-M_1x02_P7.20mm_Vertical"
 			(at 307.34 160.655 0)
 			(effects
@@
 			)
 		)
-		(property "Footprint" "Connector_AMASS:AMASS_XT60PW-M_1x02_P7.20mm_Horizontal"
+		(property "Footprint" "Connector_AMASS:AMASS_XT60-M_1x02_P7.20mm_Vertical"
 			(at 280.67 78.74 0)
 			(effects
@@
 			)
 		)
-		(property "Footprint" "Connector_AMASS:AMASS_XT60PW-M_1x02_P7.20mm_Horizontal"
+		(property "Footprint" "Connector_AMASS:AMASS_XT60-M_1x02_P7.20mm_Vertical"
 			(at 295.91 50.165 0)
 			(effects
@@
 			)
 		)
-		(property "Footprint" "Connector_AMASS:AMASS_XT60PW-M_1x02_P7.20mm_Horizontal"
+		(property "Footprint" "Connector_AMASS:AMASS_XT60-M_1x02_P7.20mm_Vertical"
 			(at 318.77 74.93 0)
 			(effects
@@
 			)
 		)
-		(property "Footprint" "Connector_AMASS:AMASS_XT60PW-M_1x02_P7.20mm_Horizontal"
+		(property "Footprint" "Connector_AMASS:AMASS_XT60-M_1x02_P7.20mm_Vertical"
 			(at 269.24 108.585 0)
 			(effects
@@
 			)
 		)
-		(property "Footprint" "Connector_AMASS:AMASS_XT60PW-M_1x02_P7.20mm_Horizontal"
+		(property "Footprint" "Connector_AMASS:AMASS_XT60-M_1x02_P7.20mm_Vertical"
 			(at 349.25 86.995 0)
 			(effects
@@
 			)
 		)
-		(property "Footprint" "Connector_AMASS:AMASS_XT60PW-M_1x02_P7.20mm_Horizontal"
+		(property "Footprint" "Connector_AMASS:AMASS_XT60-M_1x02_P7.20mm_Vertical"
 			(at 275.59 147.32 0)
 			(effects
@@
 			)
 		)
-		(property "Footprint" "Connector_AMASS:AMASS_XT60PW-M_1x02_P7.20mm_Horizontal"
+		(property "Footprint" "Connector_AMASS:AMASS_XT60-M_1x02_P7.20mm_Vertical"
 			(at 269.24 119.38 0)
 			(effects
@@
 			)
 		)
-		(property "Footprint" "Connector_AMASS:AMASS_XT60PW-M_1x02_P7.20mm_Horizontal"
+		(property "Footprint" "Connector_AMASS:AMASS_XT60-M_1x02_P7.20mm_Vertical"
 			(at 307.34 147.32 0)
 			(effects
@@
 			)
 		)
-		(property "Footprint" "Connector_AMASS:AMASS_XT60PW-M_1x02_P7.20mm_Horizontal"
+		(property "Footprint" "Connector_AMASS:AMASS_XT60-M_1x02_P7.20mm_Vertical"
 			(at 344.805 120.015 0)
 			(effects
@@
 			)
 		)
-		(property "Footprint" "Connector_AMASS:AMASS_XT60PW-M_1x02_P7.20mm_Horizontal"
+		(property "Footprint" "Connector_AMASS:AMASS_XT60-M_1x02_P7.20mm_Vertical"
 			(at 376.555 38.1 0)
 			(effects
@@
 			)
 		)
-		(property "Footprint" "Connector_AMASS:AMASS_XT60PW-M_1x02_P7.20mm_Horizontal"
+		(property "Footprint" "Connector_AMASS:AMASS_XT60-M_1x02_P7.20mm_Vertical"
 			(at 344.805 106.68 0)
 			(effects

Commit message: made a few changes in schematic
Parts:
- removed 1.5k1: 1.5k, Resistor_SMD:R_0805_2012Metric_Pad1.20x1.40mm_HandSolder, symbol Device:R_Small_US
- removed FB1: FerriteBead, PCM_Inductor_SMD_Handsoldering_AKL:L_CommonModeChoke_Coilcraft_0603USB, symbol Device:FerriteBead_Small
- removed J22: USB_C_Receptacle_USB2.0_14P, Connector_USB:USB_C_Receptacle_GCT_USB4105-xx-A_16P_TopMnt_Horizontal, symbol Connector:USB_C_Receptacle_USB2.0_14P
- removed R29, R30: 5.1k, PCM_4ms_Resistor:R_0603, symbol Device:R_US
- removed U18: USBLC6-4SC6, Package_TO_SOT_SMD:SOT-23-6, symbol Power_Protection:USBLC6-4SC6
Other:
- sheet ISOLATION & PROTRECTION renamed ISOLATION & PROTECTION
- note removed: "USB Port"
- moved on the sheet: U15
