File: base/isolation.kicad_sch (KiCad schematic)
At the start: 96 parts, among them U1 UA741CP, U10 USBLC6-4SC6, U11 USBLC6-4SC6, U2 USBLC6-4SC6, U23 6N137, U24 6N137, U25 6N137, U26 6N137, U27 6N137, U28 6N137, U29 6N137, U3 USBLC6-4SC6, U30 6N137, U31 6N137, U32 6N137, U33 6N137, U34 6N137, U36 6N137, U37 6N137

Commit message: fixed labels
Parts:
- STMCap1: footprint Connector_Phoenix_SPT:PhoenixContact_SPT_1.5_9-H-3.5_1x09_P3.5mm_Horizontal -> Capacitor_SMD:C_0805_2012Metric
Changed lines of the file:
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@@
 			)
 		)
-		(property "Footprint" "Connector_Phoenix_SPT:PhoenixContact_SPT_1.5_9-H-3.5_1x09_P3.5mm_Horizontal"
+		(property "Footprint" "Capacitor_SMD:C_0805_2012Metric"
 			(at 345.44 162.8648 0)
 			(effects

Commit message: suggested corrections made
Parts:
- removed R46, R47, R48, R49, R54, R55, R56, R57, R62, R63, R64, R65, R71, R72: 4.7k, Resistor_SMD:R_0805_2012Metric_Pad1.20x1.40mm_HandSolder, symbol Device:R
- added STMFuse2: Polyfuse, Fuse:Fuse_0603_1608Metric_Pad1.05x0.95mm_HandSolder, symbol Device:Polyfuse
Connections:
- net 3V3S is gone; now on net 5VOut: U2.5 (VBUS), U3.5 (VBUS)
- net Chassis is gone; now on net GND: H5.1, H6.1, H7.1, H8.1
- net Earth is gone; now on net GND: U10.2 (GND), U11.2 (GND), U2.2 (GND), U3.2 (GND)
- net 5VIn: now also U23.2 (A), U24.2 (A), U27.2 (A), U28.2 (A), U31.2 (A), U32.2 (A); no longer C2.1, Encoder1Capacitor1.1, Encoder1Capacitor2.1, Encoder1Capacitor3.1, L2.1
- net STM5V_ISO: now also U25.2 (A), U26.2 (A), U29.2 (A), U30.2 (A), U33.2 (A), U34.2 (A), U36.2 (A), U37.2 (A), STMFuse2.2
- net 12V_OUT_ARM renamed 12VOUT
- net 3V3M renamed 5VOut
- net 5VOut: now also C2.1, Encoder1Capacitor1.1, Encoder1Capacitor2.1, Encoder1Capacitor3.1, L2.1
- net 5V renamed STM5V_ISO_IN
- net STM5V_ISO_IN: now also STMFuse2.1
Other:
- note removed: "TVS DIODE"
- moved on the sheet: BNO1, MainFuse1

Commit message: added 0603 footprint
Parts:
- BNOCapacitor1, C2, C20, C21, C22, C23, C24, C25, C26, C27, C28, C29, C3, C30, C31, C35, C36, C5, C7, C9, Encoder1Capacitor1, Encoder1Capacitor2, Encoder1Capacitor3: footprint Capacitor_SMD:C_0805_2012Metric_Pad1.18x1.45mm_HandSolder -> Capacitor_SMD:C_0201_0603Metric
- BNOLED1, Battery_Indication2, STMLED1: footprint LED_SMD:LED_0805_2012Metric_Pad1.15x1.40mm_HandSolder -> LED_SMD:LED_0201_0603Metric
- L2: footprint Inductor_SMD:L_0805_2012Metric_Pad1.05x1.20mm_HandSolder -> PCM_Inductor_SMD_Handsoldering_AKL:L_0603_1608Metric_Pad1.05x0.95mm
- MainLED1: footprint LED_THT:LED_D3.0mm -> LED_SMD:LED_0201_0603Metric
- R10, R11, R18, R19, R20, R21, R4, R50, R51, R52, R53, R58, R59, R60, R61, R66, R67, R68, R69, R7, R73, R74, R8, R9: footprint Resistor_SMD:R_0805_2012Metric_Pad1.20x1.40mm_HandSolder -> PCM_4ms_Resistor:R_0603
- STMCap1: footprint Capacitor_SMD:C_0805_2012Metric -> Capacitor_SMD:C_0201_0603Metric

Commit message: dff
Other:
- note added: "OCTOCOUPLER"
- note removed: "OCTOCUPPLER"
Changed lines of the file:
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@@
 		)
 	)
-	(text "OCTOCUPPLER\n"
+	(text "OCTOCOUPLER\n"
 		(exclude_from_sim no)
-		(at 134.62 15.875 0)
+		(at 133.985 16.51 0)
 		(effects
 			(font

Commit message: made a few changes in schematic
Connections:
- net 5VIn: no longer C22.1, C23.1, C26.1, C27.1, C30.1, C31.1, C35.1, C36.1, R52.2, R53.2, R60.2, R61.2, R68.2, R69.2, R73.2, R74.2, U23.2 (A), U24.2 (A), U25.8 (VCC), U26.8 (VCC), U27.2 (A), U28.2 (A), U29.8 (VCC), U30.8 (VCC), U31.2 (A), U32.2 (A), U33.8 (VCC), U34.8 (VCC), U36.8 (VCC), U37.8 (VCC)
- net 5VOut: now also C22.1, C23.1, C26.1, C27.1, C30.1, C31.1, C35.1, C36.1, R52.2, R53.2, R60.2, R61.2, R68.2, R69.2, R73.2, R74.2, U23.2 (A), U24.2 (A), U25.8 (VCC), U26.8 (VCC), U27.2 (A), U28.2 (A), U29.8 (VCC), U30.8 (VCC), U31.2 (A), U32.2 (A), U33.8 (VCC), U34.8 (VCC), U36.8 (VCC), U37.8 (VCC)
- no-connect marks 39 -> 40
Other:
- note added: "ISOLATED BUCK"
- note removed: "BUCK"
- moved on the sheet: C27, R61

Commit message: new schematic
Parts:
- removed C27, C28, C29, C30, C31, C35, C36: 0.1µ, Capacitor_SMD:C_0201_0603Metric, symbol Device:C
- removed R61, R66, R67, R68, R69, R73, R74: 330, PCM_4ms_Resistor:R_0603, symbol Device:R
- removed U30, U31, U32, U33, U34, U36, U37: 6N137, Package_DIP:DIP-8_W7.62mm, symbol Isolator:6N137
- U23, U24, U25, U26, U27, U28, U29: symbol Isolator:6N137 -> Isolator:VO4661
Connections:
- net 5VOut: no longer U25.8 (VCC), U26.8 (VCC), U29.8 (VCC)
- net Encoder1AOUT: no longer U23.6 (VO)
- net Encoder1BOUT: no longer U24.6 (VO)
- net Encoder2AOUT: no longer U27.6 (VO)
- net Encoder2BOUT: no longer U28.6 (VO)
- net GND: no longer U25.5 (GND), U26.5 (GND), U29.5 (GND)
- net GND1: no longer U23.5 (GND), U24.5 (GND), U27.5 (GND), U28.5 (GND)
- net MDD1DIR: no longer U26.6 (VO)
- net MDD1PWM: no longer U25.6 (VO)
- net MDD2PWM: no longer U29.6 (VO)
- net STM5V_ISO: no longer U23.8 (VCC), U24.8 (VCC), U27.8 (VCC), U28.8 (VCC)
- no-connect marks 40 -> 22
