File: base/RCUP_BASE_PCB_2.kicad_pcb (KiCad board)
At the start: 2 copper layers, 188 x 152.4 mm, 94 parts, among them J1 MAIN KILL SWITCH, J10 ARM KILL SWITCH, J11 ISOLATED BUCK IN, J12 ISOLATED BUCK OUT, J13 JETSON BUCK IN, J14 JETSON BUCK OUT, J15 JETSON KILL SWITCH, J16 24V TO 12V BUCK, J17 24V TO 12V BUCK, J18 JETSON POWER, J19 12V_BUCK_PINOUTS_ARM, J2 MOTOR 1 PWR, J20 BatteryIN, J21 12V_BUCK_PINOUTS_ARM, J22 12V_BUCK_PINOUTS_ARM, J23 12V_BUCK_PINOUTS_ARM, J24 STEPPER AND BLDC POWER, J25 STEPPER AND BLDC POWER, J26 STEPPER AND BLDC POWER, J27 STEPPER AND BLDC POWER, J28 12V_BUCK_PINOUTS_ARM, J29 12V_BUCK_PINOUTS_ARM, J3 MOTOR 3 PWR, J30 ISOLATED STM POWER, J31 STM 2 POWER, J32 Conn_01x20_Pin, J33 Conn_01x20_Pin, J34 Conn_01x20_Pin, J35 Conn_01x20_Pin, J36 ARM KILL SWITCH 12V, J4 MOTOR 2 PWR, J40 EXTRA 12V PORT, J41 EXTRA 5V PORT, J42 EXTRA 24V PORT, J43 EXTRA 24V PORT, J5 MOTOR 4 PWR, J6 BASE KILL SWITCH 12V, J7 BASE KILL SWITCH 24V, J8 BUCK JST OUT, J9 BUCK JST IN, U1 UA741CP, U10 USBLC6-4SC6, U11 USBLC6-4SC6, U2 USBLC6-4SC6, U3 USBLC6-4SC6, U4 USBLC6-4SC6, U5 BNO055

Commit message: 50% routing done
Parts:
- removed J12: ISOLATED BUCK OUT, Connector_AMASS:AMASS_XT60-M_1x02_P7.20mm_Vertical
- removed the J13 at (222.2, 25.4)
- removed the J14 at (236.2, 25.4)
- removed the J15 at (112.2, 25.0)
- removed the J20 at (152.7, 45.3)
- removed the J25 at (194.3, 25.0)
- removed the J26 at (229.0, 102.3)
- removed the J27 at (229.0, 88.5)
- removed the J28 at (166.5, 45.3)
- removed the J29 at (180.3, 45.3)
- removed J43: EXTRA 24V PORT, Connector_AMASS:AMASS_XT60-M_1x02_P7.20mm_Vertical
- removed MainFuse1: Fuse, Fuse:Fuseholder_Littelfuse_445_030_series_5x30mm
- added H5: MountingHole_Pad, MountingHole:MountingHole_4.3mm_M4_DIN965_Pad_TopBottom, F.Cu at (60.2, 23.4)
- added H6: MountingHole_Pad, MountingHole:MountingHole_4.3mm_M4_DIN965_Pad_TopBottom, F.Cu at (60.2, 32.5)
- added H7: MountingHole_Pad, MountingHole:MountingHole_4.3mm_M4_DIN965_Pad_TopBottom, F.Cu at (60.2, 41.5)
- added H8: MountingHole_Pad, MountingHole:MountingHole_4.3mm_M4_DIN965_Pad_TopBottom, F.Cu at (60.2, 50.6)
- BNO1, U4: moved to B.Cu
- C1: renamed from C4; footprint Capacitor_SMD:C_0201_0603Metric -> Capacitor_SMD:C_0603_1608Metric_Pad1.08x0.95mm_HandSolder
- C2: footprint Capacitor_SMD:C_0201_0603Metric -> Capacitor_SMD:C_0603_1608Metric_Pad1.08x0.95mm_HandSolder
- C3: renamed from C9; footprint Capacitor_SMD:C_0201_0603Metric -> Capacitor_SMD:C_0603_1608Metric_Pad1.08x0.95mm_HandSolder
- C4: renamed from C3; footprint Capacitor_SMD:C_0201_0603Metric -> Capacitor_SMD:C_0603_1608Metric_Pad1.08x0.95mm_HandSolder
- C5: footprint Capacitor_SMD:C_0201_0603Metric -> Capacitor_SMD:C_0603_1608Metric_Pad1.08x0.95mm_HandSolder; moved to B.Cu
- C6: renamed from C7; footprint Capacitor_SMD:C_0201_0603Metric -> Capacitor_SMD:C_0603_1608Metric_Pad1.08x0.95mm_HandSolder; moved to B.Cu
- D1, D2, D4: footprint LED_SMD:LED_0201_0603Metric -> Diode_SMD:D_0805_2012Metric_Pad1.15x1.40mm_HandSolder
- J10: renamed from J1; footprint Connector_AMASS:AMASS_XT60-M_1x02_P7.20mm_Vertical -> ROBO:xt60
- J11: value ISOLATED BUCK IN -> BatteryIN; footprint Connector_AMASS:AMASS_XT60-M_1x02_P7.20mm_Vertical -> ROBO:xt60
- J13: renamed from J4; footprint Connector_AMASS:AMASS_XT60-M_1x02_P7.20mm_Vertical -> ROBO:xt60
- J14: renamed from J5; footprint Connector_AMASS:AMASS_XT60-M_1x02_P7.20mm_Vertical -> ROBO:xt60
- J15: renamed from J8; value BUCK JST OUT -> 24V TO 5V BUCK IN; footprint Connector_AMASS:AMASS_XT60-M_1x02_P7.20mm_Vertical -> ROBO:xt60
- J16: renamed from J6; footprint Connector_AMASS:AMASS_XT60-M_1x02_P7.20mm_Vertical -> ROBO:xt60
- J17: renamed from J7; footprint Connector_AMASS:AMASS_XT60-M_1x02_P7.20mm_Vertical -> ROBO:xt60
- J18: renamed from J16; value 24V TO 12V BUCK -> 24V TO 12V BUCK IN; footprint Connector_AMASS:AMASS_XT60-M_1x02_P7.20mm_Vertical -> ROBO:xt60
- J19: value 12V_BUCK_PINOUTS_ARM -> COOLING SYSTEM; footprint Connector_AMASS:AMASS_XT60-M_1x02_P7.20mm_Vertical -> ROBO:xt60
- J20: renamed from J21; value 12V_BUCK_PINOUTS_ARM -> COOLING SYSTEM; footprint Connector_AMASS:AMASS_XT60-M_1x02_P7.20mm_Vertical -> ROBO:xt60
- J21: renamed from J9; value BUCK JST IN -> 24V TO 5V BUCK OUT; footprint Connector_AMASS:AMASS_XT60-M_1x02_P7.20mm_Vertical -> ROBO:xt60
- J22: renamed from J17; value 24V TO 12V BUCK -> 24V TO 12V BUCK OUT; footprint Connector_AMASS:AMASS_XT60-M_1x02_P7.20mm_Vertical -> ROBO:xt60
- J23: renamed from J36; footprint Connector_AMASS:AMASS_XT60-M_1x02_P7.20mm_Vertical -> ROBO:xt60
- J24: renamed from J10; footprint Connector_AMASS:AMASS_XT60-M_1x02_P7.20mm_Vertical -> ROBO:xt60
- J25: renamed from J22; value 12V_BUCK_PINOUTS_ARM -> COOLING SYSTEM; footprint Connector_AMASS:AMASS_XT60-M_1x02_P7.20mm_Vertical -> ROBO:xt60
- J26: renamed from J23; value 12V_BUCK_PINOUTS_ARM -> COOLING SYSTEM; footprint Connector_AMASS:AMASS_XT60-M_1x02_P7.20mm_Vertical -> ROBO:xt60
- J27: renamed from J40; footprint Connector_AMASS:AMASS_XT60-M_1x02_P7.20mm_Vertical -> ROBO:xt60
- J28: renamed from J41; footprint Connector_AMASS:AMASS_XT60-M_1x02_P7.20mm_Vertical -> ROBO:xt60
- J29: renamed from J42; footprint Connector_AMASS:AMASS_XT60-M_1x02_P7.20mm_Vertical -> ROBO:xt60
- J30: value ISOLATED STM POWER -> Conn_01x03_Pin; footprint Connector_AMASS:AMASS_XT60-M_1x02_P7.20mm_Vertical -> Connector_JST:JST_XH_B3B-XH-A_1x03_P2.50mm_Vertical
- J31: value STM 2 POWER -> Conn_01x03_Pin; footprint Connector_AMASS:AMASS_XT60-M_1x02_P7.20mm_Vertical -> Connector_JST:JST_XH_B3B-XH-AM_1x03_P2.50mm_Vertical
- J6: renamed from J2; footprint Connector_AMASS:AMASS_XT60-M_1x02_P7.20mm_Vertical -> ROBO:xt60
- J7: renamed from J3; footprint Connector_AMASS:AMASS_XT60-M_1x02_P7.20mm_Vertical -> ROBO:xt60
- J8: renamed from J24; footprint Connector_AMASS:AMASS_XT60-M_1x02_P7.20mm_Vertical -> ROBO:xt60
- J9: renamed from J18; footprint Connector_AMASS:AMASS_XT60-M_1x02_P7.20mm_Vertical -> ROBO:xt60
- R1, R11, R12, R13, R14, R15, R16, R2, R3, R4, R6: footprint PCM_4ms_Resistor:R_0603 -> PCM_Resistor_SMD_AKL:R_0603_1608Metric_Pad0.98x0.95mm_HandSolder
- R10: renamed from R8; footprint PCM_4ms_Resistor:R_0603 -> PCM_Resistor_SMD_AKL:R_0603_1608Metric_Pad0.98x0.95mm_HandSolder; moved to B.Cu
- R17: renamed from R20; footprint PCM_4ms_Resistor:R_0603 -> PCM_Resistor_SMD_AKL:R_0603_1608Metric_Pad0.98x0.95mm_HandSolder
- R18: renamed from R22; footprint PCM_4ms_Resistor:R_0603 -> PCM_Resistor_SMD_AKL:R_0603_1608Metric_Pad0.98x0.95mm_HandSolder
- R19: renamed from R17; footprint PCM_4ms_Resistor:R_0603 -> PCM_Resistor_SMD_AKL:R_0603_1608Metric_Pad0.98x0.95mm_HandSolder; moved to B.Cu
- R20: renamed from R18; footprint PCM_4ms_Resistor:R_0603 -> PCM_Resistor_SMD_AKL:R_0603_1608Metric_Pad0.98x0.95mm_HandSolder; moved to B.Cu
- R5, R7: footprint PCM_4ms_Resistor:R_0603 -> PCM_Resistor_SMD_AKL:R_0603_1608Metric_Pad0.98x0.95mm_HandSolder; moved to B.Cu
- R8: renamed from R21; footprint PCM_4ms_Resistor:R_0603 -> PCM_Resistor_SMD_AKL:R_0603_1608Metric_Pad0.98x0.95mm_HandSolder
- R9: renamed from R23; footprint PCM_4ms_Resistor:R_0603 -> PCM_Resistor_SMD_AKL:R_0603_1608Metric_Pad0.98x0.95mm_HandSolder
- U5: renamed from U2; moved to B.Cu
- U6: renamed from U3; moved to B.Cu
- U7: renamed from U10; moved to B.Cu
- U8: renamed from U11; moved to B.Cu
- moved MDD3 189.8 mm to (237.1, 31.7), turned to -90 degrees
- moved MDD4 186.2 mm to (237.2, 56.6), turned to -90 degrees
- moved MDD1 184.2 mm to (237.1, 19.6), turned to -90 degrees
- moved MDD2 181.6 mm to (237.1, 44.0), turned to -90 degrees
- moved U3 174.9 mm to (238.3, 67.8), turned to -90 degrees
- moved BNO1 166.5 mm to (229.1, 77.7), turned to 90 degrees
- moved R20 150.5 mm to (222.5, 83.1), turned to 90 degrees
- moved J23 141.6 mm to (134.3, 157.1)
- moved J11 136.6 mm to (108.9, 21.0), turned to 0 degrees
- moved J20 133.6 mm to (108.6, 154.9), turned to 0 degrees
- moved J26 133.5 mm to (182.9, 157.5)
- moved R19 125.6 mm to (222.4, 78.1), turned to 90 degrees
- moved J25 125.4 mm to (108.6, 142.2), turned to 0 degrees
- moved J24 115.5 mm to (108.6, 83.8), turned to 0 degrees
- moved J27 110.3 mm to (232.2, 156.0)
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- renumbered Encoder4 to Encoder1, Encoder5 to Encoder2, Encoder6 to Encoder3, J32 to J1, J33 to J2, J34 to J3, J35 to J4, L2 to L1, MDD5 to MDD1, MDD6 to MDD2, MDD7 to MDD3, MDD8 to MDD4, OC3 to OC2, U9 to U2, U5 to U3
Connections:
- C4 pad 1: 5V_NON_ISO -> 5V
- C5 pad 1: Net-(U9--vin) -> Net-(U2-+vin)
- C6 pad 1: Net-(U9-Cs) -> Net-(U2-Cs)
- J3 pad 13: M3DIR -> M2DIR
- J3 pad 18: 5V -> 5V_NON_ISO_IN
- J30 pad 1: (no net) -> GND
- J30 pad 2: (no net) -> 12V
- J31 pad 1: (no net) -> GND
- J31 pad 2: (no net) -> 12V
- J4 pad 1: 5V_NON_ISO -> 5V_NON_ISO_IN
- J4 pad 10: M2DIR -> M3DIR
- J4 pad 11: unconnected-(J35-Pin_11-Pad11) -> M4DIR
- J4 pad 12: M3PWM -> unconnected-(J4-Pin_12-Pad12)
- J4 pad 13: unconnected-(J35-Pin_13-Pad13) -> M3PWM
- J4 pad 7: ENC3B -> unconnected-(J4-Pin_7-Pad7)
- J4 pad 8: ENC3A -> ENC3B
- J4 pad 9: M4DIR -> ENC3A
- L1 pad 2: Net-(U9--vin) -> Net-(U2-+vin)
- MotorController2 pad 1: 5V_NON_ISO -> 5V_NON_ISO_IN
- MotorController2 pad 10: M2DIR -> M3DIR
- MotorController2 pad 11: unconnected-(J35-Pin_11-Pad11) -> M4DIR
- MotorController2 pad 12: M3PWM -> unconnected-(J4-Pin_12-Pad12)
- MotorController2 pad 13: unconnected-(J35-Pin_13-Pad13) -> M3PWM
- MotorController2 pad 33: M3DIR -> M2DIR
- MotorController2 pad 38: 5V -> 5V_NON_ISO_IN
- MotorController2 pad 7: ENC3B -> unconnected-(J4-Pin_7-Pad7)
- MotorController2 pad 8: ENC3A -> ENC3B
- MotorController2 pad 9: M4DIR -> ENC3A
- OC1 pad 8: 5V_NON_ISO -> 5V
- R12 pad 1: ENC1A -> ENC1B
- R17 pad 1: 5V_NON_ISO -> 5V
- R18 pad 1: 5V_NON_ISO -> 5V
- R4 pad 2: Net-(R4-Pad2) -> Net-(U1-IN+)
- R6 pad 1: Net-(R4-Pad2) -> Net-(U1-IN+)
- STMFuse2 pad 1: STM5V_ISO_IN -> 5V
- STMFuse2 pad 2: STM5V_ISO -> 5V_NON_ISO_IN
- U1 pad 1: (no net) -> unconnected-(U1-OFFSET_N1-Pad1)
- U1 pad 2: (no net) -> Net-(U1-IN-)
- U1 pad 3: (no net) -> Net-(U1-IN+)
- U1 pad 4: (no net) -> GND
- U1 pad 5: (no net) -> unconnected-(U1-OFFSET_N2-Pad5)
- U1 pad 6: (no net) -> Net-(U1-OUT)
- U1 pad 7: (no net) -> 12V
- U1 pad 8: (no net) -> unconnected-(U1-NC-Pad8)
- U2 pad 5: (no net) -> 5V_ISO
- U2 pad 6: (no net) -> GND1
- U2 pad 7: (no net) -> Net-(U2-Cs)
Routing:
- net 5V: track 0.00 -> 169.6 mm
- net 5V_ISO: track 0.00 -> 161.9 mm, vias 0 -> 4
- net Net-(D2-A): track 0.00 -> 82.3 mm, vias 0 -> 2
- net STM1_TX: track 0.00 -> 66.2 mm
- net M1DIR: track 0.00 -> 63.3 mm, vias 0 -> 3
- net ENC1A: track 0.00 -> 60.2 mm, vias 0 -> 1
- net M4DIR: track 0.00 -> 59.7 mm, vias 0 -> 3
- net STM1_RX: track 0.00 -> 58.4 mm
- net M1PWM: track 0.00 -> 57.1 mm, vias 0 -> 1
- net M3PWM: track 0.00 -> 56.7 mm
- net M2DIR: track 0.00 -> 54.9 mm, vias 0 -> 3
- net M3DIR: track 0.00 -> 53.6 mm, vias 0 -> 2
- net STM2_TX: track 0.00 -> 48.4 mm, vias 0 -> 2
- net M2PWM: track 0.00 -> 48.3 mm, vias 0 -> 1
- net M4PWM: track 0.00 -> 45.9 mm, vias 0 -> 1
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- added copper zone on F.Cu, net 24V
- added copper zone on F.Cu, net 24V_BATTERY
- added copper zone on B.Cu, net GND1
- added copper zone on F.Cu, net GND1
Other:
- board size 188 x 152.4 mm -> 147.3 x 152.4 mm

Commit message: 1st iteration complete
Parts:
- J31: footprint Connector_JST:JST_XH_B3B-XH-AM_1x03_P2.50mm_Vertical -> Connector_JST:JST_XH_B3B-XH-A_1x03_P2.50mm_Vertical
- moved J15 48.6 mm to (108.6, 128.5)
- moved J19 48.6 mm to (154.4, 112.3)
- moved J27 31.5 mm to (200.7, 156.0)
- moved J28 31.5 mm to (232.2, 156.0)
- moved J13 25.1 mm to (108.6, 83.8)
- moved J24 25.1 mm to (133.7, 84.3)
- moved J17 15.2 mm to (132.6, 112.3)
- moved J8 15.2 mm to (132.6, 97.0)
Connections:
- C1 pad 2: GND -> GND1
- J15 pad N: 24V_BASE -> GND
- J15 pad P: GND -> 24V_BASE
- J27 pad P: 12V -> 12V_BASE
- J29 pad N: 24V -> GND
- J29 pad P: GND -> 24V
- J30 pad 2: 12V -> 12V_ARM
- J31 pad 2: 12V -> 12V_ARM
Routing:
- net 5V: track 169.6 -> 366.2 mm, vias 0 -> 7
- net GND1: track 20.5 -> 126.5 mm, vias 0 -> 2
- net 12V: track 0.00 -> 84.6 mm
- net 5V_NON_ISO_IN: track 23.4 -> 106.9 mm
- net ENC2B: track 35.1 -> 104.2 mm, vias 0 -> 3
- net ENC2A: track 37.1 -> 99.7 mm, vias 0 -> 3
- net ENC3A: track 27.5 -> 76.7 mm, vias 0 -> 3
- net 12V_BASE: track 0.00 -> 49.2 mm
- net 24V: track 0.00 -> 49.0 mm, vias 0 -> 2
- net 5V_ISO: track 161.9 -> 208.0 mm, vias 4 -> 6
- net BNO_SDA: track 29.1 -> 74.3 mm
- net ENC3B: track 31.9 -> 76.1 mm, vias 1 -> 3
- net BNO_SCL: track 22.3 -> 55.1 mm, vias 0 -> 2
- net ENC1B: track 22.8 -> 55.4 mm, vias 0 -> 1
- net ENC1A: track 60.2 -> 91.2 mm, vias 1 -> 2
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- added copper zone on F.Cu, net 12V
- added copper zone on B.Cu, net 12V_ARM
- added copper zone on B.Cu, net 24V
- added copper zone on F.Cu, net 24V_ARM
- added copper zone on F.Cu, net 24V_BASE
- added copper zone on B.Cu, net 24V_BATTERY
- added copper zone on B.Cu, net GND
- added copper zone on F.Cu, net GND

Commit message: 2nd iteration 50% done
Parts:
- added JP1: SolderJumper_2_Open, Jumper:SolderJumper-2_P1.3mm_Open_RoundedPad1.0x1.5mm, F.Cu at (1.68, 1.27)
- added JP2: SolderJumper_2_Open, Jumper:SolderJumper-2_P1.3mm_Open_RoundedPad1.0x1.5mm, F.Cu at (1.68, 4.83)
- J1, J2, J3, J4: footprint Connector_PinHeader_2.54mm:PinHeader_1x20_P2.54mm_Vertical_SMD_Pin1Left -> Connector_PinHeader_2.54mm:PinHeader_1x20_P2.54mm_Vertical
- R11, R12, R13, R14, R15, R16, R2, STMFuse2: moved to B.Cu
- moved H5 165.9 mm to (204.8, 104.6)
- moved H8 144.7 mm to (204.8, 54.6)
- moved H6 119.0 mm to (154.8, 104.6)
- moved H7 95.6 mm to (154.8, 54.6)
- moved J22 88.4 mm to (164.4, 69.8), turned to 0 degrees
- moved J28 74.4 mm to (164.4, 125.2), turned to 0 degrees
- moved J27 68.8 mm to (164.4, 97.5), turned to 0 degrees
- moved J16 68.5 mm to (144.0, 92.4), turned to 0 degrees
- moved C6 61.8 mm to (235.8, 106.1), turned to 180 degrees
- moved R2 60.7 mm to (230.0, 106.2), turned to -90 degrees
- moved R12 58.7 mm to (216.5, 28.6), turned to 90 degrees
- moved Encoder1 57.7 mm to (187.0, 78.6)
- moved Encoder2 57.6 mm to (187.0, 94.2)
- moved J8 56.9 mm to (173.0, 57.0), turned to 180 degrees
- moved J21 56.7 mm to (164.4, 139.0), turned to 0 degrees
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Connections:
- J1 pad 18: 5V_ISO -> Net-(J1-Pin_18)
- J2 pad 1: 5V_ISO_FUSE_OUT -> Net-(J2-Pin_1)
- MotorController1 pad 1: 5V_ISO_FUSE_OUT -> Net-(J2-Pin_1)
- MotorController1 pad 38: 5V_ISO -> Net-(J1-Pin_18)
Routing:
- net 5V: track 366.2 -> 0.00 mm, vias 7 -> 0
- net 5V_ISO: track 208.0 -> 0.00 mm, vias 6 -> 0
- net GND1: track 126.5 -> 0.00 mm, vias 2 -> 0
- net ENC2B: track 104.2 -> 7.62 mm, vias 3 -> 0
- net ENC2A: track 99.7 -> 7.62 mm, vias 3 -> 0
- net 5V_NON_ISO_IN: track 106.9 -> 15.2 mm
- net 12V: track 84.6 -> 0.00 mm
- net ENC1A: track 91.2 -> 7.62 mm, vias 2 -> 0
- net Net-(D2-A): track 82.3 -> 0.00 mm, vias 2 -> 0
- net ENC3A: track 76.7 -> 7.62 mm, vias 3 -> 0
- net ENC3B: track 76.1 -> 7.62 mm, vias 3 -> 0
- net BNO_SDA: track 74.3 -> 7.62 mm
- net STM1_TX: track 66.2 -> 7.62 mm
- net M1DIR: track 63.3 -> 7.62 mm, vias 3 -> 0
- net 5V_ISO_FUSE_OUT: track 54.5 -> 0.00 mm, vias 3 -> 0
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- added copper zone on B.Cu, net 12V
- added copper zone on B.Cu, net 24V_ARM
- added copper zone on B.Cu, net 24V_BASE
- removed copper zone on B.Cu, net 12V_ARM
Other:
- board size 147.3 x 152.4 mm -> 128 x 133.4 mm

Commit message: 2nd iteration done
Parts:
- C4: moved to B.Cu
- L1: footprint PCM_Inductor_SMD_Handsoldering_AKL:L_0603_1608Metric_Pad1.05x0.95mm -> footprints:IND_SWPA5040S_SNL-M
- moved JP2 261.8 mm to (231.7, 130.0), turned to -90 degrees
- moved JP1 215.0 mm to (182.0, 118.3), turned to 90 degrees
- moved R12 27.9 mm to (188.8, 31.8)
- moved L1 2.25 mm to (223.1, 95.8)
- moved C4 1.13 mm to (197.2, 66.2)
- moved C5 0.08 mm to (223.1, 106.1)
Connections:
- C1 pad 1: 5V_ISO_FUSE_OUT -> 5V_ISO
- H5 pad 1: Chassis -> GND
- H6 pad 1: Chassis -> GND
- H7 pad 1: Chassis -> GND
- H8 pad 1: Chassis -> GND
- OC2 pad 8: 5V_ISO_FUSE_OUT -> 5V_ISO
- R8 pad 1: 5V_ISO_FUSE_OUT -> 5V_ISO
- R9 pad 1: 5V_ISO_FUSE_OUT -> 5V_ISO
Routing:
- net GND: track 7.62 -> 243.8 mm, vias 0 -> 23
- net 5V: track 0.00 -> 223.8 mm, vias 0 -> 16
- net 5V_ISO: track 0.00 -> 186.2 mm, vias 0 -> 12
- net Net-(D2-A): track 0.00 -> 118.2 mm, vias 0 -> 1
- net BNO_SDA: track 7.62 -> 121.2 mm, vias 0 -> 2
- net GND1: track 0.00 -> 101.3 mm, vias 0 -> 5
- net ENC2A: track 7.62 -> 105.7 mm, vias 0 -> 3
- net STM1_TX: track 7.62 -> 105.6 mm
- net M4DIR: track 7.62 -> 104.1 mm, vias 0 -> 3
- net 5V_NON_ISO_IN: track 15.2 -> 106.8 mm
- net ENC2B: track 7.62 -> 97.7 mm, vias 0 -> 2
- net STM1_RX: track 7.62 -> 79.5 mm, vias 0 -> 2
- net ENC1A: track 7.62 -> 75.3 mm, vias 0 -> 3
- net M3DIR: track 7.62 -> 75.1 mm, vias 0 -> 3
- net M3PWM: track 7.62 -> 70.7 mm, vias 0 -> 4
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- added copper zone on B.Cu, net 12V_ARM
- added copper zone on F.Cu, net 12V_ARM
Other:
- board size 128 x 133.4 mm -> 126.2 x 133.1 mm

Commit message: 2nd iteration fixed
Parts:
- removed D3: 1N47xxA, Diode_THT:D_DO-41_SOD81_P10.16mm_Horizontal
- removed D4: LED, Diode_SMD:D_0805_2012Metric_Pad1.15x1.40mm_HandSolder
- removed R10: 1k, PCM_Resistor_SMD_AKL:R_0603_1608Metric_Pad0.98x0.95mm_HandSolder
- removed R3: 410, PCM_Resistor_SMD_AKL:R_0603_1608Metric_Pad0.98x0.95mm_HandSolder
- removed R4: 620, PCM_Resistor_SMD_AKL:R_0603_1608Metric_Pad0.98x0.95mm_HandSolder
- removed R5, R6, R7: 10K, PCM_Resistor_SMD_AKL:R_0603_1608Metric_Pad0.98x0.95mm_HandSolder
- removed U1: UA741CP, UA741CP:DIP794W45P254L959H508Q8
- moved OC2 11.4 mm to (201.0, 75.5), turned to 0 degrees
Routing:
- net GND: track 243.8 -> 195.8 mm, vias 23 -> 1136
- net 12V: track 39.5 -> 0.00 mm, vias 2 -> 0
- net Net-(D3-K): track 34.9 -> 0.00 mm, vias 1 -> 0
- net Net-(D4-A): track 29.6 -> 0.00 mm, vias 1 -> 0
- net Net-(U1-IN+): track 18.6 -> 0.00 mm, vias 1 -> 0
- net 24V: track 44.5 -> 27.3 mm, vias 2 -> 109
- net Net-(OC2-Pad2): track 4.21 -> 19.9 mm, vias 0 -> 2
- net 5V_ISO: track 186.2 -> 175.1 mm
- net STM2_TX: track 48.8 -> 58.7 mm, vias 1 -> 2
- net Net-(U1-IN-): track 9.84 -> 0.00 mm, vias 1 -> 0
- net Net-(U1-OUT): track 7.88 -> 0.00 mm
- net GND1: track 101.3 -> 97.8 mm, vias 5 -> 102
- net Net-(D2-A): track 118.2 -> 121.4 mm
- net 5V_ISO_BNO: track 13.6 -> 14.7 mm
- net STM1_RX: track 79.5 -> 79.6 mm, vias 2 -> 3
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