File: base/untitled.kicad_sch (KiCad schematic)
At the start: 37 parts, among them J10 MAIN KILL SWITCH, J11 BatteryIN, J13 MOTOR 2 PWR, J14 MOTOR 4 PWR, J15 24V TO 5V BUCK IN, J16 BASE KILL SWITCH 12V, J17 BASE KILL SWITCH 24V, J18 24V TO 12V BUCK IN, J19 COOLING SYSTEM, J20 COOLING SYSTEM, J21 24V TO 5V BUCK OUT, J22 24V TO 12V BUCK OUT, J23 ARM KILL SWITCH 12V, J24 ARM KILL SWITCH, J25 COOLING SYSTEM, J26 COOLING SYSTEM, J27 EXTRA 12V PORT, J28 EXTRA 5V PORT, J29 EXTRA 24V PORT, J30 Conn_01x03_Pin, J31 Conn_01x03_Pin, J6 MOTOR 1 PWR, J7 MOTOR 3 PWR, J8 STEPPER AND BLDC POWER, J9 JETSON POWER, U4 USBLC6-4SC6, U5 USBLC6-4SC6, U6 USBLC6-4SC6, U7 USBLC6-4SC6, U8 USBLC6-4SC6

Commit message: 2nd iteration 50% done
Connections:
- net 12V: no longer J27.P (POS)
- net 12V_BASE: now also J27.P (POS)
Other:
- moved on the sheet: H5, H6, H7, H8
Changed lines of the file:
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@@
 	)
 	(rectangle
-		(start 218.44 144.78)
-		(end 271.145 179.07)
+		(start 200.025 127)
+		(end 252.73 161.29)
 		(stroke
 			(width 0.381)
@@
 	(text "Mounting Holes\n"
 		(exclude_from_sim no)
-		(at 244.475 143.51 0)
+		(at 226.06 125.73 0)
 		(effects
 			(font
@@
 	(text_box "Mounting holes for earthing are used to connect the PCB’s ground plane to the chassis or metal enclosure, providing a safety discharge path and reducing EMI (electromagnetic interference)."
 		(exclude_from_sim no)
-		(at 224.155 163.83 0)
+		(at 205.74 146.05 0)
 		(size 41.275 11.43)
 		(margins 0.9525 0.9525 0.9525 0.9525)
@@
 		)
 	)
+	(global_label "12V_BASE"
+		(shape input)
+		(at 180.34 31.75 180)
+		(fields_autoplaced yes)
+		(effects
+			(font
+				(size 1.27 1.27)
+			)
+			(justify right)
+		)
+		(property "Intersheetrefs" "${INTERSHEET_REFS}"
+			(at 168.1625 31.75 0)
+			(effects
+				(font
+					(size 1.27 1.27)
+				)
+				(justify right)
+				(hide yes)
+			)
+		)
+	)
 	(global_label "M4DIR"
 		(shape input)
@@
 		)
 	)
-	(global_label "12V"
-		(shape input)
-		(at 180.34 31.75 180)
-		(fields_autoplaced yes)
-		(effects
-			(font
-				(size 1.27 1.27)
-			)
-			(justify right)
-		)
-		(property "Intersheetrefs" "${INTERSHEET_REFS}"
-			(at 173.8472 31.75 0)
-			(effects
-				(font
-					(size 1.27 1.27)
-				)
-				(justify right)
-				(hide yes)
-			)
-		)
-	)
 	(global_label "24V"
 		(shape input)
@@
 	(symbol
 		(lib_id "power:GNDPWR")
-		(at 251.46 154.305 0)
+		(at 233.045 136.525 0)
 		(unit 1)
 		(exclude_from_sim no)
@@
 		(dnp no)
 		(property "Reference" "#PWR051"
-			(at 251.46 160.655 0)
+			(at 233.045 142.875 0)
 			(effects
 				(font
@@
 		)
 		(property "Value" "Chassis"
-			(at 250.698 153.035 0)
+			(at 232.283 135.255 0)
 			(effects
 				(font
@@
 		)
 		(property "Footprint" ""
-			(at 251.46 155.575 0)
+			(at 233.045 137.795 0)
 			(effects
 				(font
@@
 		)
 		(property "Datasheet" "~"
-			(at 251.46 155.575 0)
+			(at 233.045 137.795 0)
 			(effects
 				(font
@@
 		)
 		(property "Description" "Power symbol creates a global label with name \"GNDPWR\" , global ground"
-			(at 251.46 154.305 0)
+			(at 233.045 136.525 0)
 			(effects
 				(font
@@
 	(symbol
 		(lib_id "Mechanical:MountingHole_Pad")
-		(at 238.76 151.765 0)
+		(at 220.345 133.985 0)
 		(unit 1)
 		(exclude_from_sim yes)
@@
 		(fields_autoplaced yes)
 		(property "Reference" "H6"
-			(at 241.3 149.2249 0)
+			(at 222.885 131.4449 0)
 			(effects
 				(font
@@
 		)
 		(property "Value" "MountingHole_Pad"
-			(at 241.3 151.7649 0)
+			(at 222.885 133.9849 0)
 			(effects
 				(font
@@
 		)
 		(property "Footprint" "MountingHole:MountingHole_4.3mm_M4_DIN965_Pad_TopBottom"
-			(at 238.76 151.765 0)
+			(at 220.345 133.985 0)
 			(effects
 				(font
@@
 		)
 		(property "Datasheet" "~"
-			(at 238.76 151.765 0)
+			(at 220.345 133.985 0)
 			(effects
 				(font
@@
 		)
 		(property "Description" "Mounting Hole with connection"
-			(at 238.76 151.765 0)
+			(at 220.345 133.985 0)
 			(effects
 				(font
@@
 	(symbol
 		(lib_id "Mechanical:MountingHole_Pad")
-		(at 262.89 151.765 0)
+		(at 244.475 133.985 0)
 		(unit 1)
 		(exclude_from_sim yes)
@@
 		(fields_autoplaced yes)
 		(property "Reference" "H8"
-			(at 265.43 149.2249 0)
+			(at 247.015 131.4449 0)
 			(effects
 				(font
@@
 		)
 		(property "Value" "MountingHole_Pad"
-			(at 265.43 151.7649 0)
+			(at 247.015 133.9849 0)
 			(effects
 				(font
@@
 		)
 		(property "Footprint" "MountingHole:MountingHole_4.3mm_M4_DIN965_Pad_TopBottom"
-			(at 262.89 151.765 0)
+			(at 244.475 133.985 0)
 			(effects
 				(font
@@
 		)
 		(property "Datasheet" "~"
-			(at 262.89 151.765 0)
+			(at 244.475 133.985 0)
 			(effects
 				(font
@@
 		)
 		(property "Description" "Mounting Hole with connection"
-			(at 262.89 151.765 0)
+			(at 244.475 133.985 0)
 			(effects
 				(font
@@
 	(symbol
 		(lib_id "power:GNDPWR")
-		(at 238.76 154.305 0)
+		(at 220.345 136.525 0)
 		(unit 1)
 		(exclude_from_sim no)
@@
 		(dnp no)
 		(property "Reference" "#PWR050"
-			(at 238.76 160.655 0)
+			(at 220.345 142.875 0)
 			(effects
 				(font
@@
 		)
 		(property "Value" "Chassis"
-			(at 237.998 153.035 0)
+			(at 219.583 135.255 0)
 			(effects
 				(font
@@
 		)
 		(property "Footprint" ""
-			(at 238.76 155.575 0)
+			(at 220.345 137.795 0)
 			(effects
 				(font
@@
 		)
 		(property "Datasheet" "~"
-			(at 238.76 155.575 0)
+			(at 220.345 137.795 0)
 			(effects
 				(font
@@
 		)
 		(property "Description" "Power symbol creates a global label with name \"GNDPWR\" , global ground"
-			(at 238.76 154.305 0)
+			(at 220.345 136.525 0)
 			(effects
 				(font
@@
 	(symbol
 		(lib_id "power:GNDPWR")
-		(at 226.06 154.305 0)
+		(at 207.645 136.525 0)
 		(unit 1)
 		(exclude_from_sim no)
@@
 		(dnp no)
 		(property "Reference" "#PWR049"
-			(at 226.06 160.655 0)
+			(at 207.645 142.875 0)
 			(effects
 				(font
@@
 		)
 		(property "Value" "Chassis"
-			(at 225.298 153.035 0)
+			(at 206.883 135.255 0)
 			(effects
 				(font
@@
 		)
 		(property "Footprint" ""
-			(at 226.06 155.575 0)
+			(at 207.645 137.795 0)
 			(effects
 				(font
@@
 		)
 		(property "Datasheet" "~"
-			(at 226.06 155.575 0)
+			(at 207.645 137.795 0)
 			(effects
 				(font
@@
 		)
 		(property "Description" "Power symbol creates a global label with name \"GNDPWR\" , global ground"
-			(at 226.06 154.305 0)
+			(at 207.645 136.525 0)
 			(effects
 				(font
@@
 	(symbol
 		(lib_id "power:GNDPWR")
-		(at 262.89 154.305 0)
+		(at 244.475 136.525 0)
 		(unit 1)
 		(exclude_from_sim no)
@@
 		(dnp no)
 		(property "Reference" "#PWR052"
-			(at 262.89 160.655 0)
+			(at 244.475 142.875 0)
 			(effects
 				(font
@@
 		)
 		(property "Value" "Chassis"
-			(at 262.128 153.035 0)
+			(at 243.713 135.255 0)
 			(effects
 				(font
@@
 		)
 		(property "Footprint" ""
-			(at 262.89 155.575 0)
+			(at 244.475 137.795 0)
 			(effects
 				(font
@@
 		)
 		(property "Datasheet" "~"
-			(at 262.89 155.575 0)
+			(at 244.475 137.795 0)
 			(effects
 				(font
@@
 		)
 		(property "Description" "Power symbol creates a global label with name \"GNDPWR\" , global ground"
-			(at 262.89 154.305 0)
+			(at 244.475 136.525 0)
 			(effects
 				(font
@@
 	(symbol
 		(lib_id "Mechanical:MountingHole_Pad")
-		(at 226.06 151.765 0)
+		(at 207.645 133.985 0)
 		(unit 1)
 		(exclude_from_sim yes)
@@
 		(fields_autoplaced yes)
 		(property "Reference" "H5"
-			(at 228.6 149.2249 0)
+			(at 210.185 131.4449 0)
 			(effects
 				(font
@@
 		)
 		(property "Value" "MountingHole_Pad"
-			(at 228.6 151.7649 0)
+			(at 210.185 133.9849 0)
 			(effects
 				(font
@@
 		)
 		(property "Footprint" "MountingHole:MountingHole_4.3mm_M4_DIN965_Pad_TopBottom"
-			(at 226.06 151.765 0)
+			(at 207.645 133.985 0)
 			(effects
 				(font
@@
 		)
 		(property "Datasheet" "~"
-			(at 226.06 151.765 0)
+			(at 207.645 133.985 0)
 			(effects
 				(font
@@
 		)
 		(property "Description" "Mounting Hole with connection"
-			(at 226.06 151.765 0)
+			(at 207.645 133.985 0)
 			(effects
 				(font
@@
 	(symbol
 		(lib_id "Mechanical:MountingHole_Pad")
-		(at 251.46 151.765 0)
+		(at 233.045 133.985 0)
 		(unit 1)
 		(exclude_from_sim yes)
@@
 		(fields_autoplaced yes)
 		(property "Reference" "H7"
-			(at 254 149.2249 0)
+			(at 235.585 131.4449 0)
 			(effects
 				(font
@@
 		)
 		(property "Value" "MountingHole_Pad"
-			(at 254 151.7649 0)
+			(at 235.585 133.9849 0)
 			(effects
 				(font
@@
 		)
 		(property "Footprint" "MountingHole:MountingHole_4.3mm_M4_DIN965_Pad_TopBottom"
-			(at 251.46 151.765 0)
+			(at 233.045 133.985 0)
 			(effects
 				(font
@@
 		)
 		(property "Datasheet" "~"
-			(at 251.46 151.765 0)
+			(at 233.045 133.985 0)
 			(effects
 				(font
@@
 		)
 		(property "Description" "Mounting Hole with connection"
-			(at 251.46 151.765 0)
+			(at 233.045 133.985 0)
 			(effects
 				(font

Commit message: 2nd iteration fixed
Connections:
- net Chassis is gone; now on net GND: H5.1, H6.1, H7.1, H8.1
Changed lines of the file:
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@@
 	)
 	(symbol
-		(lib_id "power:GNDPWR")
+		(lib_id "power:GND")
 		(at 233.045 136.525 0)
 		(unit 1)
@@
 		(on_board yes)
 		(dnp no)
-		(property "Reference" "#PWR051"
+		(fields_autoplaced yes)
+		(property "Reference" "#PWR049"
 			(at 233.045 142.875 0)
 			(effects
@@
 			)
 		)
-		(property "Value" "Chassis"
-			(at 232.283 135.255 0)
+		(property "Value" "GND"
+			(at 233.045 140.97 0)
 			(effects
 				(font
@@
 		)
 		(property "Footprint" ""
-			(at 233.045 137.795 0)
+			(at 233.045 136.525 0)
 			(effects
 				(font
@@
 			)
 		)
-		(property "Datasheet" "~"
-			(at 233.045 137.795 0)
+		(property "Datasheet" ""
+			(at 233.045 136.525 0)
 			(effects
 				(font
@@
 			)
 		)
-		(property "Description" "Power symbol creates a global label with name \"GNDPWR\" , global ground"
+		(property "Description" "Power symbol creates a global label with name \"GND\" , ground"
 			(at 233.045 136.525 0)
 			(effects
@@
 		)
 		(instances
-			(project "RCUP_BASE_PCB_2"
+			(project ""
 				(path "/926cf7a2-92fe-4b49-b65d-bdeab2e766b1/fe4912c4-5108-4cc8-bf1b-0fd11e27f186"
-					(reference "#PWR051")
+					(reference "#PWR049")
 					(unit 1)
 				)
@@
 	(symbol
 		(lib_id "power:GND")
+		(at 220.345 136.525 0)
+		(unit 1)
+		(exclude_from_sim no)
+		(in_bom yes)
+		(on_board yes)
+		(dnp no)
+		(fields_autoplaced yes)
+		(property "Reference" "#PWR050"
+			(at 220.345 142.875 0)
+			(effects
+				(font
+					(size 1.27 1.27)
+				)
+				(hide yes)
+			)
+		)
+		(property "Value" "GND"
+			(at 220.345 140.97 0)
+			(effects
+				(font
+					(size 1.27 1.27)
+				)
+			)
+		)
+		(property "Footprint" ""
+			(at 220.345 136.525 0)
+			(effects
+				(font
+					(size 1.27 1.27)
+				)
+				(hide yes)
+			)
+		)
+		(property "Datasheet" ""
+			(at 220.345 136.525 0)
+			(effects
+				(font
+					(size 1.27 1.27)
+				)
+				(hide yes)
+			)
+		)
+		(property "Description" "Power symbol creates a global label with name \"GND\" , ground"
+			(at 220.345 136.525 0)
+			(effects
+				(font
+					(size 1.27 1.27)
+				)
+				(hide yes)
+			)
+		)
+		(pin "1"
+		)
+		(instances
+			(project ""
+				(path "/926cf7a2-92fe-4b49-b65d-bdeab2e766b1/fe4912c4-5108-4cc8-bf1b-0fd11e27f186"
+					(reference "#PWR050")
+					(unit 1)
+				)
+			)
+		)
+	)
+	(symbol
+		(lib_id "power:GND")
 		(at 119.507 110.998 0)
 		(unit 1)
@@
 	)
 	(symbol
+		(lib_id "power:GND")
+		(at 207.645 136.525 0)
+		(unit 1)
+		(exclude_from_sim no)
+		(in_bom yes)
+		(on_board yes)
+		(dnp no)
+		(fields_autoplaced yes)
+		(property "Reference" "#PWR051"
+			(at 207.645 142.875 0)
+			(effects
+				(font
+					(size 1.27 1.27)
+				)
+				(hide yes)
+			)
+		)
+		(property "Value" "GND"
+			(at 207.645 140.97 0)
+			(effects
+				(font
+					(size 1.27 1.27)
+				)
+			)
+		)
+		(property "Footprint" ""
+			(at 207.645 136.525 0)
+			(effects
+				(font
+					(size 1.27 1.27)
+				)
+				(hide yes)
+			)
+		)
+		(property "Datasheet" ""
+			(at 207.645 136.525 0)
+			(effects
+				(font
+					(size 1.27 1.27)
+				)
+				(hide yes)
+			)
+		)
+		(property "Description" "Power symbol creates a global label with name \"GND\" , ground"
+			(at 207.645 136.525 0)
+			(effects
+				(font
+					(size 1.27 1.27)
+				)
+				(hide yes)
+			)
+		)
+		(pin "1"
+		)
+		(instances
+			(project ""
+				(path "/926cf7a2-92fe-4b49-b65d-bdeab2e766b1/fe4912c4-5108-4cc8-bf1b-0fd11e27f186"
+					(reference "#PWR051")
+					(unit 1)
+				)
+			)
+		)
+	)
+	(symbol
 		(lib_id "XT60-M:XT60-M")
 		(at 185.42 34.29 0)
@@
 	)
 	(symbol
-		(lib_id "power:GNDPWR")
-		(at 220.345 136.525 0)
-		(unit 1)
-		(exclude_from_sim no)
-		(in_bom yes)
-		(on_board yes)
-		(dnp no)
-		(property "Reference" "#PWR050"
-			(at 220.345 142.875 0)
-			(effects
-				(font
-					(size 1.27 1.27)
-				)
-				(hide yes)
-			)
-		)
-		(property "Value" "Chassis"
-			(at 219.583 135.255 0)
-			(effects
-				(font
-					(size 1.27 1.27)
-				)
-			)
-		)
-		(property "Footprint" ""
-			(at 220.345 137.795 0)
-			(effects
-				(font
-					(size 1.27 1.27)
-				)
-				(hide yes)
-			)
-		)
-		(property "Datasheet" "~"
-			(at 220.345 137.795 0)
-			(effects
-				(font
-					(size 1.27 1.27)
-				)
-				(hide yes)
-			)
-		)
-		(property "Description" "Power symbol creates a global label with name \"GNDPWR\" , global ground"
-			(at 220.345 136.525 0)
-			(effects
-				(font
-					(size 1.27 1.27)
-				)
-				(hide yes)
-			)
-		)
-		(pin "1"
-		)
-		(instances
-			(project "RCUP_BASE_PCB_2"
-				(path "/926cf7a2-92fe-4b49-b65d-bdeab2e766b1/fe4912c4-5108-4cc8-bf1b-0fd11e27f186"
-					(reference "#PWR050")
-					(unit 1)
-				)
-			)
-		)
-	)
-	(symbol
 		(lib_id "Connector:Conn_01x03_Pin")
 		(at 58.42 134.62 0)
@@
 	)
 	(symbol
-		(lib_id "power:GNDPWR")
-		(at 207.645 136.525 0)
-		(unit 1)
-		(exclude_from_sim no)
-		(in_bom yes)
-		(on_board yes)
-		(dnp no)
-		(property "Reference" "#PWR049"
-			(at 207.645 142.875 0)
-			(effects
-				(font
-					(size 1.27 1.27)
-				)
-				(hide yes)
-			)
-		)
-		(property "Value" "Chassis"
-			(at 206.883 135.255 0)
-			(effects
-				(font
-					(size 1.27 1.27)
-				)
-			)
-		)
-		(property "Footprint" ""
-			(at 207.645 137.795 0)
-			(effects
-				(font
-					(size 1.27 1.27)
-				)
-				(hide yes)
-			)
-		)
-		(property "Datasheet" "~"
-			(at 207.645 137.795 0)
-			(effects
-				(font
-					(size 1.27 1.27)
-				)
-				(hide yes)
-			)
-		)
-		(property "Description" "Power symbol creates a global label with name \"GNDPWR\" , global ground"
-			(at 207.645 136.525 0)
-			(effects
-				(font
-					(size 1.27 1.27)
-				)
-				(hide yes)
-			)
-		)
-		(pin "1"
-		)
-		(instances
-			(project "RCUP_BASE_PCB_2"
-				(path "/926cf7a2-92fe-4b49-b65d-bdeab2e766b1/fe4912c4-5108-4cc8-bf1b-0fd11e27f186"
-					(reference "#PWR049")
-					(unit 1)
-				)
-			)
-		)
-	)
-	(symbol
 		(lib_id "XT60-M:XT60-M")
 		(at 124.587 97.663 0)
@@
 	)
 	(symbol
-		(lib_id "power:GNDPWR")
-		(at 244.475 136.525 0)
-		(unit 1)
-		(exclude_from_sim no)
-		(in_bom yes)
-		(on_board yes)
-		(dnp no)
-		(property "Reference" "#PWR052"
-			(at 244.475 142.875 0)
-			(effects
-				(font
-					(size 1.27 1.27)
-				)
-				(hide yes)
-			)
-		)
-		(property "Value" "Chassis"
-			(at 243.713 135.255 0)
-			(effects
-				(font
-					(size 1.27 1.27)
-				)
-			)
-		)
-		(property "Footprint" ""
-			(at 244.475 137.795 0)
-			(effects
-				(font
-					(size 1.27 1.27)
-				)
-				(hide yes)
-			)
-		)
-		(property "Datasheet" "~"
-			(at 244.475 137.795 0)
-			(effects
-				(font
-					(size 1.27 1.27)
-				)
-				(hide yes)
-			)
-		)
-		(property "Description" "Power symbol creates a global label with name \"GNDPWR\" , global ground"
-			(at 244.475 136.525 0)
-			(effects
-				(font
-					(size 1.27 1.27)
-				)
-				(hide yes)
-			)
-		)
-		(pin "1"
-		)
-		(instances
-			(project "RCUP_BASE_PCB_2"
-				(path "/926cf7a2-92fe-4b49-b65d-bdeab2e766b1/fe4912c4-5108-4cc8-bf1b-0fd11e27f186"
-					(reference "#PWR052")
-					(unit 1)
-				)
-			)
-		)
-	)
-	(symbol
 		(lib_id "Device:Polyfuse")
 		(at 121.92 139.065 90)
@@
 					(unit 1)
 				)
+			)
+		)
+	)
+	(symbol
+		(lib_id "power:GND")
+		(at 244.475 136.525 0)
+		(unit 1)
+		(exclude_from_sim no)
+		(in_bom yes)
+		(on_board yes)
+		(dnp no)
+		(fields_autoplaced yes)
+		(property "Reference" "#PWR033"
+			(at 244.475 142.875 0)
+			(effects
+				(font
+					(size 1.27 1.27)
+				)
+				(hide yes)
+			)
+		)
+		(property "Value" "GND"
+			(at 244.475 140.97 0)
+			(effects
+				(font
+					(size 1.27 1.27)
+				)
+			)
+		)
+		(property "Footprint" ""
+			(at 244.475 136.525 0)
+			(effects
+				(font
+					(size 1.27 1.27)
+				)
+				(hide yes)
+			)
+		)
+		(property "Datasheet" ""
+			(at 244.475 136.525 0)
+			(effects
+				(font
+					(size 1.27 1.27)
+				)
+				(hide yes)
+			)
+		)
+		(property "Description" "Power symbol creates a global label with name \"GND\" , ground"
+			(at 244.475 136.525 0)
+			(effects
+				(font
+					(size 1.27 1.27)
+				)
+				(hide yes)
+			)
+		)
+		(pin "1"
+		)
+		(instances
+			(project ""
+				(path "/926cf7a2-92fe-4b49-b65d-bdeab2e766b1/fe4912c4-5108-4cc8-bf1b-0fd11e27f186"
+					(reference "#PWR033")
+					(unit 1)
+				)
