File: base/untitled.kicad_sch (KiCad schematic)
At the start: 37 parts, among them J10 MAIN KILL SWITCH, J11 BatteryIN, J13 MOTOR 2 PWR, J14 MOTOR 4 PWR, J15 24V TO 5V BUCK IN, J16 BASE KILL SWITCH 12V, J17 BASE KILL SWITCH 24V, J18 24V TO 12V BUCK IN, J19 COOLING SYSTEM, J20 COOLING SYSTEM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

Commit message: fixed all the previous issues added mpu footprint
Connections:
- net 5V_NON_ISO_IN renamed 5V_NON_ISO_FUSE_OUT
Other:
- moved on the sheet: J28, J30, J31, STMFuse2
