File: base/RCUP_BASE_PCB_2.kicad_sch (KiCad schematic)
At the start: 49 parts, among them J1 Conn_01x20_Pin, J2 Conn_01x20_Pin, J3 Conn_01x20_Pin, J4 Conn_01x20_Pin, U1 UA741CP, U3 BNO055

Commit message: 2nd iteration 50% done
Parts:
- added JP1, JP2: SolderJumper_2_Open, Jumper:SolderJumper-2_P1.3mm_Open_RoundedPad1.0x1.5mm, symbol Jumper:SolderJumper_2_Open
- J1, J2, J3, J4: footprint Connector_PinHeader_2.54mm:PinHeader_1x20_P2.54mm_Vertical_SMD_Pin1Left -> Connector_PinHeader_2.54mm:PinHeader_1x20_P2.54mm_Vertical
Connections:
- net 5V_ISO: now also JP2.1 (A); no longer J1.18 (Pin_18), MotorController1.38 (5V)
- net 5V_ISO_FUSE_OUT: now also JP1.2 (B); no longer J2.1 (Pin_1), MotorController1.1 (5V)
- new net: J1.18 (Pin_18), JP2.2 (B), MotorController1.38 (5V)
- new net: J2.1 (Pin_1), JP1.1 (A), MotorController1.1 (5V)
Other:
- sheet p renamed Ports
Changed lines of the file:
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@@
 	(wire
 		(pts
-			(xy 76.2 22.225) (xy 67.31 22.225)
+			(xy 83.185 22.225) (xy 88.9 22.225)
 		)
 		(stroke
@@
 	(wire
 		(pts
+			(xy 75.565 22.225) (xy 67.31 22.225)
+		)
+		(stroke
+			(width 0)
+			(type default)
+		)
+	)
+	(wire
+		(pts
 			(xy 142.875 144.145) (xy 144.145 144.145)
 		)
@@
 	(wire
 		(pts
+			(xy 37.465 65.405) (xy 45.72 65.405)
+		)
+		(stroke
+			(width 0)
+			(type default)
+		)
+	)
+	(wire
+		(pts
 			(xy 150.495 182.245) (xy 149.225 182.245)
 		)
@@
 	(wire
 		(pts
-			(xy 39.37 65.405) (xy 45.72 65.405)
+			(xy 27.94 65.405) (xy 29.845 65.405)
 		)
 		(stroke
@@
 	(global_label "5V_ISO"
 		(shape input)
-		(at 39.37 65.405 180)
+		(at 27.94 65.405 180)
 		(fields_autoplaced yes)
 		(effects
@@
 		)
 		(property "Intersheetrefs" "${INTERSHEET_REFS}"
-			(at 29.9743 65.405 0)
+			(at 18.5443 65.405 0)
 			(effects
 				(font
@@
 	(global_label "5V_ISO_FUSE_OUT"
 		(shape input)
-		(at 76.2 22.225 0)
+		(at 88.9 22.225 0)
 		(fields_autoplaced yes)
 		(effects
@@
 		)
 		(property "Intersheetrefs" "${INTERSHEET_REFS}"
-			(at 95.9371 22.225 0)
+			(at 108.6371 22.225 0)
 			(effects
 				(font
@@
 			)
 		)
-		(property "Footprint" "Connector_PinHeader_2.54mm:PinHeader_1x20_P2.54mm_Vertical_SMD_Pin1Left"
+		(property "Footprint" "Connector_PinHeader_2.54mm:PinHeader_1x20_P2.54mm_Vertical"
 			(at 247.65 45.72 0)
 			(effects
@@
 	)
 	(symbol
+		(lib_id "Jumper:SolderJumper_2_Open")
+		(at 33.655 65.405 0)
+		(unit 1)
+		(exclude_from_sim no)
+		(in_bom no)
+		(on_board yes)
+		(dnp no)
+		(fields_autoplaced yes)
+		(property "Reference" "JP2"
+			(at 33.655 59.69 0)
+			(effects
+				(font
+					(size 1.27 1.27)
+				)
+			)
+		)
+		(property "Value" "SolderJumper_2_Open"
+			(at 33.655 62.23 0)
+			(effects
+				(font
+					(size 1.27 1.27)
+				)
+			)
+		)
+		(property "Footprint" "Jumper:SolderJumper-2_P1.3mm_Open_RoundedPad1.0x1.5mm"
+			(at 33.655 65.405 0)
+			(effects
+				(font
+					(size 1.27 1.27)
+				)
+				(hide yes)
+			)
+		)
+		(property "Datasheet" "~"
+			(at 33.655 65.405 0)
+			(effects
+				(font
+					(size 1.27 1.27)
+				)
+				(hide yes)
+			)
+		)
+		(property "Description" "Solder Jumper, 2-pole, open"
+			(at 33.655 65.405 0)
+			(effects
+				(font
+					(size 1.27 1.27)
+				)
+				(hide yes)
+			)
+		)
+		(pin "1"
+		)
+		(pin "2"
+		)
+		(instances
+			(project ""
+				(path "/926cf7a2-92fe-4b49-b65d-bdeab2e766b1"
+					(reference "JP2")
+					(unit 1)
+				)
+			)
+		)
+	)
+	(symbol
 		(lib_id "Connector:Conn_01x03_Pin")
 		(at 43.18 177.165 0)
@@
 	(symbol
 		(lib_id "power:GND1")
-		(at 99.06 24.765 180)
+		(at 99.06 24.765 0)
 		(unit 1)
 		(exclude_from_sim no)
@@
 		(fields_autoplaced yes)
 		(property "Reference" "#PWR011"
-			(at 99.06 18.415 0)
+			(at 99.06 31.115 0)
 			(effects
 				(font
@@
 		)
 		(property "Value" "GND1"
-			(at 99.06 20.32 0)
+			(at 101.6 26.0349 0)
 			(effects
 				(font
 					(size 1.27 1.27)
 				)
+				(justify left)
 			)
 		)
@@
 			)
 		)
-		(property "Footprint" "Connector_PinHeader_2.54mm:PinHeader_1x20_P2.54mm_Vertical_SMD_Pin1Left"
+		(property "Footprint" "Connector_PinHeader_2.54mm:PinHeader_1x20_P2.54mm_Vertical"
 			(at 72.39 45.085 0)
 			(effects
@@
 			)
 		)
-		(property "Footprint" "Connector_PinHeader_2.54mm:PinHeader_1x20_P2.54mm_Vertical_SMD_Pin1Left"
+		(property "Footprint" "Connector_PinHeader_2.54mm:PinHeader_1x20_P2.54mm_Vertical"
 			(at 215.9 45.72 0)
 			(effects
@@
 			)
 		)
-		(property "Footprint" "Connector_PinHeader_2.54mm:PinHeader_1x20_P2.54mm_Vertical_SMD_Pin1Left"
+		(property "Footprint" "Connector_PinHeader_2.54mm:PinHeader_1x20_P2.54mm_Vertical"
 			(at 40.64 45.085 0)
 			(effects
@@
 	)
 	(symbol
+		(lib_id "Jumper:SolderJumper_2_Open")
+		(at 79.375 22.225 0)
+		(unit 1)
+		(exclude_from_sim no)
+		(in_bom no)
+		(on_board yes)
+		(dnp no)
+		(fields_autoplaced yes)
+		(property "Reference" "JP1"
+			(at 79.375 16.51 0)
+			(effects
+				(font
+					(size 1.27 1.27)
+				)
+			)
+		)
+		(property "Value" "SolderJumper_2_Open"
+			(at 79.375 19.05 0)
+			(effects
+				(font
+					(size 1.27 1.27)
+				)
+			)
+		)
+		(property "Footprint" "Jumper:SolderJumper-2_P1.3mm_Open_RoundedPad1.0x1.5mm"
+			(at 79.375 22.225 0)
+			(effects
+				(font
+					(size 1.27 1.27)
+				)
+				(hide yes)
+			)
+		)
+		(property "Datasheet" "~"
+			(at 79.375 22.225 0)
+			(effects
+				(font
+					(size 1.27 1.27)
+				)
+				(hide yes)
+			)
+		)
+		(property "Description" "Solder Jumper, 2-pole, open"
+			(at 79.375 22.225 0)
+			(effects
+				(font
+					(size 1.27 1.27)
+				)
+				(hide yes)
+			)
+		)
+		(pin "1"
+		)
+		(pin "2"
+		)
+		(instances
+			(project ""
+				(path "/926cf7a2-92fe-4b49-b65d-bdeab2e766b1"
+					(reference "JP1")
+					(unit 1)
+				)
+			)
+		)
+	)
+	(symbol
 		(lib_id "Device:R_Small_US")
 		(at 187.96 151.13 90)
@@
 			(color 0 0 0 0.0000)
 		)
-		(property "Sheetname" "p"
+		(property "Sheetname" "Ports"
 			(at 219.71 113.665 0)
 			(effects

Commit message: 2nd iteration fixed
Parts:
- removed D3: 1N47xxA, Diode_THT:D_DO-41_SOD81_P10.16mm_Horizontal, symbol Diode:1N47xxA
- removed D4: LED, Diode_SMD:D_0805_2012Metric_Pad1.15x1.40mm_HandSolder, symbol Device:LED
- removed R10: 1k, PCM_Resistor_SMD_AKL:R_0603_1608Metric_Pad0.98x0.95mm_HandSolder, symbol Device:R_Small_US
- removed R3: 410, PCM_Resistor_SMD_AKL:R_0603_1608Metric_Pad0.98x0.95mm_HandSolder, symbol Device:R_Small_US
- removed R4: 620, PCM_Resistor_SMD_AKL:R_0603_1608Metric_Pad0.98x0.95mm_HandSolder, symbol Device:R_Small_US
- removed R5, R6, R7: 10K, PCM_Resistor_SMD_AKL:R_0603_1608Metric_Pad0.98x0.95mm_HandSolder, symbol Device:R_Small_US
- removed U1: UA741CP, UA741CP:DIP794W45P254L959H508Q8, symbol ROBO misc symbols:uA741CP
- L1: footprint PCM_Inductor_SMD_Handsoldering_AKL:L_0603_1608Metric_Pad1.05x0.95mm -> footprints:IND_SWPA5040S_SNL-M
Connections:
- net 5V_ISO: now also C1.1, OC2.8 (VCC), R8.1, R9.1
- net 5V_ISO_FUSE_OUT: no longer C1.1, OC2.8 (VCC), R8.1, R9.1
- no-connect marks 60 -> 57
Other:
- note removed: "BATTERY INDICATOR"

Commit message: fixed dfm errors some still left
Parts:
- C5: footprint Capacitor_SMD:C_0603_1608Metric_Pad1.08x0.95mm_HandSolder -> Capacitor_Tantalum_SMD:CP_EIA-3216-18_Kemet-A_HandSolder
- C6: footprint Capacitor_SMD:C_0603_1608Metric_Pad1.08x0.95mm_HandSolder -> PCM_Capacitor_Tantalum_SMD_AKL:CP_EIA-6032-28_Kemet-C_Pad2.25x2.35mm_HandSolder
Changed lines of the file:
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@@
 			)
 		)
-		(property "Footprint" "Capacitor_SMD:C_0603_1608Metric_Pad1.08x0.95mm_HandSolder"
+		(property "Footprint" "Capacitor_Tantalum_SMD:CP_EIA-3216-18_Kemet-A_HandSolder"
 			(at 180.0352 95.885 0)
 			(effects
@@
 			)
 		)
-		(property "Footprint" "Capacitor_SMD:C_0603_1608Metric_Pad1.08x0.95mm_HandSolder"
+		(property "Footprint" "PCM_Capacitor_Tantalum_SMD_AKL:CP_EIA-6032-28_Kemet-C_Pad2.25x2.35mm_HandSolder"
 			(at 178.1048 107.95 0)
 			(effects
